Commit message: Add real cart body mesh, four casters, and headless sim runner
raskogbody.stl replaces the placeholder box on base_link, with all four
of the stock RASKOG cart's casters modeled (not just a rear pair - the
drive wheels are an addition, not a replacement for any of them).

Split the Isaac Sim ros2_control bridge into per-command-interface-type
hardware components: mixing velocity-commanded wheels with
position-commanded head joints in one component let
joint_state_topic_hardware_interface emit a JointState with mismatched
array lengths, which Isaac's ROS2SubscribeJointState rejected. Also
gives every sim joint an explicit effort state interface and initial
values, both required by controller_manager/sum_wrapped_joint_states,
not optional polish.

sim/run_headless.py is the non-GUI entry point for driving the twin
from a script or CI instead of the interactive launch_gui.py.

Also latches the teleop safety supervisor's e-stop until joint_states
actually recovers, instead of firing once and never clearing.

File: src/xlerobot_description/urdf/base_2wheels.xacro (robot description, xacro)
@@ -52,4 +52,36 @@
     </joint>
   </xacro:macro>
+  <!-- Four generic casters, not two: the stock RASKOG cart's original four
+       wheels are all still there - the drive wheels are an addition on
+       their own extended axle bar, not a replacement for any of them (see
+       the photo this was built from). A single centered caster, or just a
+       rear pair, would both be wrong - this is front pair + rear pair, all
+       four passive. No encoder on any of them, so each is a fixed sphere
+       and not a joint - a joint would just publish made up numbers. Their
+       scrub when turning in place is part of why yaw needs IMU fusion. -->
+  <xacro:macro name="caster" params="prefix reflect x_offset dims">
+    <xacro:property name="b" value="${dims['base']}"/>
+    <link name="${prefix}_caster_link">
+      <visual>
+        <geometry><sphere radius="${b['caster_radius']}"/></geometry>
+        <material name="xle_black"/>
+      </visual>
+      <collision>
+        <geometry><sphere radius="${b['caster_radius']}"/></geometry>
+        <surface><friction><ode><mu>0.05</mu><mu2>0.05</mu2></ode></friction></surface>
+      </collision>
+      <inertial>
+        <mass value="0.05"/>
+        <inertia ixx="1e-5" ixy="0" ixz="0" iyy="1e-5" iyz="0" izz="1e-5"/>
+      </inertial>
+    </link>
+    <joint name="${prefix}_caster_joint" type="fixed">
+      <parent link="base_link"/>
+      <child  link="${prefix}_caster_link"/>
+      <origin xyz="${x_offset}
+                   ${reflect * b['caster_y_offset']}
+                   ${b['caster_radius']}" rpy="0 0 0"/>
+    </joint>
+  </xacro:macro>
   <xacro:macro name="xlerobot_base" params="dims">
     <xacro:property name="b" value="${dims['base']}"/>
@@ -63,13 +95,30 @@
     <!-- base_link origin is on the floor, between the drive wheels -->
     <link name="base_link">
+      <!-- raskogbody.stl, from upstream's own Isaac Sim asset bundle
+           (Apache-2.0, simulation/Isaac_sim/xlerobot.zip), same IKEA RASKOG
+           cart this robot is built on. The offset here is derived, not
+           measured: upstream's reference URDF places this mesh at
+           xyz="-0.01668 0.502 0.515" rpy="90 0 0" relative to their own
+           "chassis" link, whose wheel joints sit at xyz="-0.15 +-0.225 -0.32"
+           and whose floor height comes from its floating joint to world
+           (z=0.38). Re-expressing that mesh offset relative to OUR base_link
+           (floor level, at the midpoint between the wheels) gives
+           xyz="0.13332 0.502 0.895" - visually verify once this is open in
+           Isaac Sim and nudge if it's off; this wasn't checked against the
+           real robot's actual proportions, only against upstream's own
+           reference numbers. Does NOT include upstream's raskogwheel1/2.stl
+           sub-meshes deliberately: those depict the stock cart's original
+           four casters at their stock 0.45m track, which is narrower than
+           this robot's actual 0.55m custom drive-wheel track (measured) -
+           including them would draw a second, wrong-width pair of wheels
+           overlapping the real ones modeled below. -->
       <visual>
-        <origin xyz="0 0 ${b['body_height']/2.0}" rpy="0 0 0"/>
+        <origin xyz="0.13332 0.502 0.895" rpy="${pi/2} 0 0"/>
         <geometry>
-          <box size="${b['body_length']} ${b['body_width']} ${b['body_height']}"/>
+          <mesh filename="package://xlerobot_description/meshes/raskogbody.stl"
+                scale="0.0009 0.001 0.0009"/>
         </geometry>
         <material name="xle_grey"/>
       </visual>
-      <!-- TODO use raskogbody.stl from the upstream Isaac Sim bundle.
-           Box is close enough for costmap work until then. -->
       <collision>
         <origin xyz="0 0 ${b['body_height']/2.0}" rpy="0 0 0"/>
@@ -91,27 +140,8 @@
     <xacro:drive_wheel prefix="left"  reflect="1"  dims="${dims}"/>
     <xacro:drive_wheel prefix="right" reflect="-1" dims="${dims}"/>
-    <!-- Caster has no encoder, so it's a fixed sphere and not a joint. A joint
-         would just publish made up numbers. Its scrub when turning in place is
-         part of why yaw needs IMU fusion. -->
-    <link name="caster_link">
-      <visual>
-        <geometry><sphere radius="${b['caster_radius']}"/></geometry>
-        <material name="xle_black"/>
-      </visual>
-      <collision>
-        <geometry><sphere radius="${b['caster_radius']}"/></geometry>
-        <surface><friction><ode><mu>0.05</mu><mu2>0.05</mu2></ode></friction></surface>
-      </collision>
-      <inertial>
-        <mass value="0.05"/>
-        <inertia ixx="1e-5" ixy="0" ixz="0" iyy="1e-5" iyz="0" izz="1e-5"/>
-      </inertial>
-    </link>
-    <joint name="caster_joint" type="fixed">
-      <parent link="base_link"/>
-      <child  link="caster_link"/>
-      <origin xyz="${b['caster_x_offset']} ${b['caster_y_offset']} ${b['caster_radius']}"
-              rpy="0 0 0"/>
-    </joint>
+    <xacro:caster prefix="rear_left"   reflect="1"  x_offset="${b['caster_rear_x_offset']}"  dims="${dims}"/>
+    <xacro:caster prefix="rear_right"  reflect="-1" x_offset="${b['caster_rear_x_offset']}"  dims="${dims}"/>
+    <xacro:caster prefix="front_left"  reflect="1"  x_offset="${b['caster_front_x_offset']}" dims="${dims}"/>
+    <xacro:caster prefix="front_right" reflect="-1" x_offset="${b['caster_front_x_offset']}" dims="${dims}"/>
   </xacro:macro>
 </robot>

File: src/xlerobot_description/urdf/xlerobot.ros2_control_sim.xacro (robot description, xacro)
@@ -27,4 +27,17 @@
        match the real robot's own ros2_control block, and the whole point
        of this twin is testing that real config, not a generic one. -->
+  <!-- effort is declared on every joint below even though Isaac Sim has no
+       real torque feedback for it: controller_manager's enforce_command_limits
+       builds a JointSaturationLimiter per joint regardless of whether that
+       joint has an effort limit, and it reads the effort state interface
+       unconditionally - without it, the read cycle throws
+       "requested state interface not found" and controller_manager
+       deactivates everything. Matches xlerobot.ros2_control.xacro's real
+       joints, which all export effort via sts_hardware_interface anyway.
+       initial_value 0.0 on effort matters here: Isaac Sim's ROS2PublishJointState
+       node doesn't populate JointState.effort, and joint_state_topic_hardware_interface
+       only calls set_state() for effort when that array is non-empty, so
+       without an explicit initial value the interface would sit at
+       ros2_control's own NaN default forever instead of a real number. -->
   <xacro:macro name="sim_position_joint" params="name initial_position:=0.0">
     <joint name="${name}">
@@ -34,4 +47,7 @@
       </state_interface>
       <state_interface name="velocity"/>
+      <state_interface name="effort">
+        <param name="initial_value">0.0</param>
+      </state_interface>
     </joint>
   </xacro:macro>
@@ -39,13 +55,48 @@
     <joint name="${name}">
       <command_interface name="velocity"/>
-      <state_interface name="position"/>
-      <state_interface name="velocity"/>
+      <!-- initial_value matters more here than it looks: sum_wrapped_joint_states
+           computes each new position as a delta against get_state()'s previous
+           value to unwrap Isaac's +-2pi convention. Without an initial_value,
+           that previous value starts at ros2_control's NaN default, the first
+           delta computation poisons it to NaN, and since the result is written
+           straight back with set_state(), every following cycle reads NaN as
+           "previous" too - a permanent stuck state, not a startup race. -->
+      <state_interface name="position">
+        <param name="initial_value">0.0</param>
+      </state_interface>
+      <state_interface name="velocity">
+        <param name="initial_value">0.0</param>
+      </state_interface>
+      <state_interface name="effort">
+        <param name="initial_value">0.0</param>
+      </state_interface>
     </joint>
   </xacro:macro>
   <xacro:macro name="xlerobot_ros2_control_sim" params="with_arms dims">
-    <ros2_control name="xlerobot_sim" type="system">
+    <!-- Split into two hardware components, one per command-interface type,
+         not one combined block like an earlier version of this file had.
+         joint_state_topic_hardware_interface's write() pushes every joint's
+         name unconditionally but only appends to position/velocity/effort
+         for the command interfaces that joint actually declares - mixing
+         velocity-commanded wheels with position-commanded head/arm joints
+         in one component produced a JointState message with a 4-entry name
+         array next to 2-entry position/velocity arrays, silently
+         misaligning the indices. Isaac Sim's ROS2SubscribeJointState node
+         correctly refuses that ("size of position, velocity and effort
+         arrays match the number of actuators") rather than guess. Keeping
+         each component homogeneous (all-velocity or all-position) means
+         its arrays are always either full-length or fully empty, which is
+         what sensor_msgs/JointState actually promises. Same reasoning as
+         the real robot's two-bus split, different underlying cause.
+         joint_states_topic (read side) stays the single shared
+         /isaac_joint_states for both: JointStateTopicSystem::read() looks
+         up each incoming name against its own joints and skips anything it
+         doesn't recognize, so one combined state message covering every
+         joint is fine to share - only the outgoing command side has the
+         strict per-array-length problem. -->
+    <ros2_control name="xlerobot_sim_wheels" type="system">
       <hardware>
         <plugin>joint_state_topic_hardware_interface/JointStateTopicSystem</plugin>
-        <param name="joint_commands_topic">/isaac_joint_commands</param>
+        <param name="joint_commands_topic">/isaac_wheel_commands</param>
         <param name="joint_states_topic">/isaac_joint_states</param>
         <param name="sum_wrapped_joint_states">true</param>
@@ -53,4 +104,12 @@
       <xacro:sim_velocity_joint name="left_wheel_joint"/>
       <xacro:sim_velocity_joint name="right_wheel_joint"/>
+    </ros2_control>
+    <ros2_control name="xlerobot_sim_position" type="system">
+      <hardware>
+        <plugin>joint_state_topic_hardware_interface/JointStateTopicSystem</plugin>
+        <param name="joint_commands_topic">/isaac_position_commands</param>
+        <param name="joint_states_topic">/isaac_joint_states</param>
+        <param name="sum_wrapped_joint_states">true</param>
+      </hardware>
       <xacro:sim_position_joint name="head_pan_joint"/>
       <xacro:sim_position_joint name="head_tilt_joint"/>

Commit message: Centre the base collision box on the cart body
The box was centred on the drive axle (x=0), but the cart body spans
x=-0.048 to 0.344, so it stuck out 0.18 m behind and stopped 0.12 m short
of the front. New body_x_offset (0.148, the centre of raskogbody.stl's
footprint) moves it onto the body. Size is unchanged, still the nominal
RASKOG dimensions.

File: src/xlerobot_description/urdf/base_2wheels.xacro (robot description, xacro)
@@ -122,5 +122,5 @@
       </visual>
       <collision>
-        <origin xyz="0 0 ${b['body_height']/2.0}" rpy="0 0 0"/>
+        <origin xyz="${b['body_x_offset']} 0 ${b['body_height']/2.0}" rpy="0 0 0"/>
         <geometry>
           <box size="${b['body_length']} ${b['body_width']} ${b['body_height']}"/>

Commit message: Front of the robot is the drive-wheel end, arms point forward
The model had the robot facing the caster end, the opposite of the real one.
Evidence that the front is the drive-wheel end: the mast axis is 70 mm from
the rim nearest the drive wheels (measured), the shared upstream URDF's head
camera faces -x and it names the arm at y<0 the left one, the arms point
forward in the official 0.4.0 assembly video, and in the recorded goal run
the head camera moved toward what it looks at, so +vx drives to the front.

base_link now has x to the front. The cart, the arms and the head keep the
shared URDF's numbers under body_link, base_link turned 180 degrees about z,
the drive wheels stay on base_link, the casters move (front pair +0.04, rear
pair -0.31). The left arm is the one at +y in base_link, the mast axis is
5.6 cm behind the axle line. Both arms point forward at the zero pose
(right_yaw and left_yaw -1.5708), the shared URDF has them sideways. The head
camera and both wrist cameras now look along +x, the head camera was looking
backwards. Nav2 footprint flipped to match, rerun_bridge camera reframed.

The Isaac Sim scene has to be regenerated for this.

File: src/xlerobot_description/urdf/base_2wheels.xacro (robot description, xacro)
@@ -93,6 +93,30 @@
       <origin xyz="0 0 0" rpy="0 0 0"/>
     </joint>
-    <!-- base_link origin is on the floor, between the drive wheels -->
+    <!-- base_link origin is on the floor, between the drive wheels, x points to
+         the front of the robot: the end with the drive wheels, where the arms
+         and the head camera face and where it drives. Only the inertial is here. -->
     <link name="base_link">
+      <!-- inertia about the real CoM, not the box centre. Cart is top heavy
+           and this is what sets the accel limits. -->
+      <inertial>
+        <origin xyz="0 0 ${b['com_height']}" rpy="0 0 0"/>
+        <mass value="${b['body_mass']}"/>
+        <inertia
+          ixx="${b['body_mass']*(b['body_width']**2 + b['body_height']**2)/12.0}" ixy="0" ixz="0"
+          iyy="${b['body_mass']*(b['body_length']**2 + b['body_height']**2)/12.0}" iyz="0"
+          izz="${b['body_mass']*(b['body_length']**2 + b['body_width']**2)/12.0}"/>
+      </inertial>
+    </link>
+    <!-- The cart, the arms and the head are described in the frame of the shared
+         upstream URDF (simulation/xlerobot/xlerobot.urdf of the XLeRobot repo),
+         where the front is -x: drive wheels at the front, casters behind. body_link
+         is that frame, base_link turned 180 degrees about z, so their numbers can
+         be used as they are. The drive wheels stay on base_link. -->
+    <joint name="body_joint" type="fixed">
+      <parent link="base_link"/>
+      <child  link="body_link"/>
+      <origin xyz="0 0 0" rpy="0 0 ${pi}"/>
+    </joint>
+    <link name="body_link">
       <!-- raskogbody.stl, from upstream's own Isaac Sim asset bundle
            (Apache-2.0, simulation/Isaac_sim/xlerobot.zip), same IKEA RASKOG
@@ -127,14 +151,4 @@
         </geometry>
       </collision>
-      <!-- inertia about the real CoM, not the box centre. Cart is top heavy
-           and this is what sets the accel limits. -->
-      <inertial>
-        <origin xyz="0 0 ${b['com_height']}" rpy="0 0 0"/>
-        <mass value="${b['body_mass']}"/>
-        <inertia
-          ixx="${b['body_mass']*(b['body_width']**2 + b['body_height']**2)/12.0}" ixy="0" ixz="0"
-          iyy="${b['body_mass']*(b['body_length']**2 + b['body_height']**2)/12.0}" iyz="0"
-          izz="${b['body_mass']*(b['body_length']**2 + b['body_width']**2)/12.0}"/>
-      </inertial>
     </link>
     <xacro:drive_wheel prefix="left"  reflect="1"  dims="${dims}"/>

File: src/xlerobot_description/urdf/xlerobot.urdf.xacro (robot description, xacro)
@@ -38,5 +38,5 @@
   <xacro:include filename="$(find xlerobot_description)/urdf/sensors.xacro"/>
   <xacro:xlerobot_base dims="${dims}"/>
-  <xacro:xlerobot_head dims="${dims}" parent="base_link"/>
+  <xacro:xlerobot_head dims="${dims}" parent="body_link"/>
   <xacro:xlerobot_sensors sensor="$(arg sensor)" dims="${dims}"/>
   <xacro:if value="$(arg with_arms)">
@@ -51,9 +51,9 @@
     <xacro:property name="a" value="${dims['arms']}"/>
     <xacro:property name="pan_off" value="0.0452"/>
-    <xacro:so101_arm prefix="left_arm"  parent="base_link"
-        xyz="${a['mount_x'] - pan_off * sin(a['left_yaw'])}  ${a['mount_y'] + pan_off * cos(a['left_yaw'])} ${a['mount_z']}"
+    <xacro:so101_arm prefix="left_arm"  parent="body_link"
+        xyz="${a['mount_x'] - pan_off * sin(a['left_yaw'])} ${-a['mount_y'] + pan_off * cos(a['left_yaw'])} ${a['mount_z']}"
         rpy="0 0 ${a['left_yaw']}"/>
-    <xacro:so101_arm prefix="right_arm" parent="base_link"
-        xyz="${a['mount_x'] - pan_off * sin(a['right_yaw'])} ${-a['mount_y'] + pan_off * cos(a['right_yaw'])} ${a['mount_z']}"
+    <xacro:so101_arm prefix="right_arm" parent="body_link"
+        xyz="${a['mount_x'] - pan_off * sin(a['right_yaw'])}  ${a['mount_y'] + pan_off * cos(a['right_yaw'])} ${a['mount_z']}"
         rpy="0 0 ${a['right_yaw']}"/>
   </xacro:if>

Commit message: Cart, head and camera positions from measurements on the robot
Top basket: front rim 22 mm ahead of the drive axle line, rear rim 260 mm
behind it, so 282 mm long, upstream's cart mesh has 325 mm. The mesh is scaled
0.868 along the robot's length and placed so the rims match, and the
casters, the collision box and the Nav2 footprint follow (casters +0.045 and
-0.259, box 0.34 long, footprint x -0.30 to +0.08). Width and height keep
upstream's scale, not measured.

Mast axis 70 mm behind the front rim, so 48 mm behind the axle line, the arm
pan axes are at the same x. Head camera lens 65 mm behind the front rim, 5 mm
ahead of the pan axis, camera_x in the yaml.

File: src/xlerobot_description/urdf/base_2wheels.xacro (robot description, xacro)
@@ -119,5 +119,10 @@
     </joint>
     <link name="body_link">
-      <!-- raskogbody.stl, from upstream's own Isaac Sim asset bundle
+      <!-- Scaled 0.868 along the robot's length (x) from upstream's 0.0009 so the top
+           basket is 282 mm front rim to rear rim, as measured on the robot, upstream's
+           mesh has 325 mm. Front rim 22 mm ahead of the drive axle line, rear rim 260 mm
+           behind it, measured. Width and height are still upstream's scale. The rest of
+           this comment is about upstream's placement.
+           raskogbody.stl, from upstream's own Isaac Sim asset bundle
            (Apache-2.0, simulation/Isaac_sim/xlerobot.zip), same IKEA RASKOG
            cart this robot is built on. The offset here is derived, not
@@ -138,8 +143,8 @@
            overlapping the real ones modeled below. -->
       <visual>
-        <origin xyz="0.13332 0.502 0.895" rpy="${pi/2} 0 0"/>
+        <origin xyz="0.10583 0.502 0.895" rpy="${pi/2} 0 0"/>
         <geometry>
           <mesh filename="package://xlerobot_description/meshes/raskogbody.stl"
-                scale="0.0009 0.001 0.0009"/>
+                scale="0.000781 0.001 0.0009"/>
         </geometry>
         <material name="xle_grey"/>

File: src/xlerobot_description/urdf/head_pantilt.xacro (robot description, xacro)
@@ -120,5 +120,5 @@
       <child link="head_camera_mount"/>
       <!-- z puts the lens centre at head: camera_z above the floor -->
-      <origin xyz="0.025 0 ${h['camera_z'] - pan_z - 0.09815}" rpy="0 0 0"/>
+      <origin xyz="${h['camera_x']} 0 ${h['camera_z'] - pan_z - 0.09815}" rpy="0 0 0"/>
     </joint>
   </xacro:macro>
