Commit message: Fix mirrored-wheel sign and bus1 crash on the real cart
Drove each wheel individually through a raw JointGroupVelocityController
(bypassing diff_drive_controller) to find out which motor is actually
mounted mirrored - it's the right one, not the left as an earlier
comment guessed from upstream's docs. sts_hardware_interface has no
per-joint invert, so the fix lives in diff_drive_controller's own
right_wheel_radius_multiplier: -1.0, which flips both the outgoing
command and the odometry reading consistently. Confirmed straight-line
driving on hardware after the change.

Also gate bus1's ros2_control component behind with_arms/with_head:
it declared head_pan/head_tilt unconditionally, so a base-only robot
with nothing plugged into bus1 took controller_manager down entirely
(two hardware components racing on the same serial fd when bus1_port
was pointed at bus2 for testing, or a hard failure opening a
nonexistent port otherwise).

xlerobot_setup_usb_modules.py now defaults new udev rules to 0666
instead of 0660+dialout, so a freshly generated rule doesn't need a
group membership change and re-login before the port is usable.

File: src/xlerobot_description/urdf/xlerobot.ros2_control.xacro (robot description, xacro)
@@ -44,31 +44,40 @@
     </joint>
   </xacro:macro>
-  <xacro:macro name="xlerobot_ros2_control" params="bus1_port bus2_port use_mock_hardware with_arms dims">
+  <xacro:macro name="xlerobot_ros2_control" params="bus1_port bus2_port use_mock_hardware with_arms with_head dims">
     <xacro:property name="b"      value="${dims['base']}"/>
     <xacro:property name="h"      value="${dims['head']}"/>
     <xacro:property name="wmax"   value="${dims['limits']['wheel_max_angular_velocity']}"/>
     <!-- ================= BUS 1 : left arm + head ================= -->
-    <ros2_control name="xlerobot_bus1" type="system">
-      <hardware>
-        <plugin>sts_hardware_interface/STSHardwareInterface</plugin>
-        <param name="serial_port">${bus1_port}</param>
-        <param name="baud_rate">1000000</param>
-        <param name="enable_mock_mode">$(arg use_mock_hardware)</param>
-      </hardware>
-      <xacro:if value="${with_arms}">
-        <!-- phase 3. Limits are placeholders, check against
-             adityakamath/so_arm_ros2 and ros-physical-ai/ros2_so_arm -->
-        <xacro:sts_position_joint name="left_arm_shoulder_pan"   id="1" lower="-3.14" upper="3.14"/>
-        <xacro:sts_position_joint name="left_arm_shoulder_lift"  id="2" lower="-1.75" upper="1.75"/>
-        <xacro:sts_position_joint name="left_arm_elbow_flex"     id="3" lower="-1.75" upper="1.75"/>
-        <xacro:sts_position_joint name="left_arm_wrist_flex"     id="4" lower="-1.75" upper="1.75"/>
-        <xacro:sts_position_joint name="left_arm_wrist_roll"     id="5" lower="-3.14" upper="3.14"/>
-        <xacro:sts_position_joint name="left_arm_gripper"        id="6" lower="0.0"   upper="1.75"/>
-      </xacro:if>
-      <xacro:sts_position_joint name="head_pan_joint"  id="7"
-                                lower="${h['pan_limit_lower']}"  upper="${h['pan_limit_upper']}"/>
-      <xacro:sts_position_joint name="head_tilt_joint" id="8"
-                                lower="${h['tilt_limit_lower']}" upper="${h['tilt_limit_upper']}"/>
-    </ros2_control>
+    <!-- Only declared when something is actually on it. Otherwise this
+         component still tries to open bus1_port for zero joints, and on a
+         base-only robot that port doesn't exist - controller_manager loads
+         all hardware components in one process, so a bad bus1_port there
+         takes bus2 (the wheels) down with it too. -->
+    <xacro:if value="${with_arms or with_head}">
+      <ros2_control name="xlerobot_bus1" type="system">
+        <hardware>
+          <plugin>sts_hardware_interface/STSHardwareInterface</plugin>
+          <param name="serial_port">${bus1_port}</param>
+          <param name="baud_rate">1000000</param>
+          <param name="enable_mock_mode">$(arg use_mock_hardware)</param>
+        </hardware>
+        <xacro:if value="${with_arms}">
+          <!-- phase 3. Limits are placeholders, check against
+               adityakamath/so_arm_ros2 and ros-physical-ai/ros2_so_arm -->
+          <xacro:sts_position_joint name="left_arm_shoulder_pan"   id="1" lower="-3.14" upper="3.14"/>
+          <xacro:sts_position_joint name="left_arm_shoulder_lift"  id="2" lower="-1.75" upper="1.75"/>
+          <xacro:sts_position_joint name="left_arm_elbow_flex"     id="3" lower="-1.75" upper="1.75"/>
+          <xacro:sts_position_joint name="left_arm_wrist_flex"     id="4" lower="-1.75" upper="1.75"/>
+          <xacro:sts_position_joint name="left_arm_wrist_roll"     id="5" lower="-3.14" upper="3.14"/>
+          <xacro:sts_position_joint name="left_arm_gripper"        id="6" lower="0.0"   upper="1.75"/>
+        </xacro:if>
+        <xacro:if value="${with_head}">
+          <xacro:sts_position_joint name="head_pan_joint"  id="7"
+                                    lower="${h['pan_limit_lower']}"  upper="${h['pan_limit_upper']}"/>
+          <xacro:sts_position_joint name="head_tilt_joint" id="8"
+                                    lower="${h['tilt_limit_lower']}" upper="${h['tilt_limit_upper']}"/>
+        </xacro:if>
+      </ros2_control>
+    </xacro:if>
     <!-- ================= BUS 2 : right arm + DRIVE WHEELS ================= -->
     <ros2_control name="xlerobot_bus2" type="system">
@@ -87,6 +96,9 @@
         <xacro:sts_position_joint name="right_arm_gripper"       id="6" lower="0.0"   upper="1.75"/>
       </xacro:if>
-      <!-- Left motor is mounted mirrored, command has to be negated, otherwise
-           x.vel turns the robot and theta.vel drives it forward.
+      <!-- The RIGHT motor is mounted mirrored (confirmed on the real robot by
+           commanding each wheel individually and watching it turn - see
+           controllers.yaml's right_wheel_radius_multiplier comment; an
+           earlier version of this comment guessed it was the left motor,
+           that guess was wrong).
            Checked the driver source: it has no per-joint invert param. What it
            does have is a FIXED, uniform CW-to-REP103-CCW inversion applied the
@@ -94,9 +106,11 @@
            problem (protocol convention) to ours (this robot's mechanical
            mounting). It doesn't help here.
-           Not solved yet. NOT in this file: don't add a fake invert param, it
-           will be silently ignored (joint.parameters.count() just won't find
-           it, no error). Real options are an upstream patch adding a per-joint
-           invert, or a small wrapper class. Left uncorrected on purpose until
-           one of those exists, see ARCHITECTURE.md section 1.2 and 7 (R1). -->
+           NOT in this file: don't add a fake invert param, it will be
+           silently ignored (joint.parameters.count() just won't find it, no
+           error). The actual fix is diff_drive_controller's
+           right_wheel_radius_multiplier: -1.0, see controllers.yaml - that's
+           the "sign goes in the ros2_control joint config, once" ARCHITECTURE.md
+           section 1.2 talks about, just one layer up from here since the
+           hardware interface itself can't do it. -->
       <joint name="left_wheel_joint">
         <param name="motor_id">9</param>

File: src/xlerobot_description/urdf/xlerobot.urdf.xacro (robot description, xacro)
@@ -25,4 +25,9 @@
   <!-- arms are phase 3, description only for now -->
   <xacro:arg name="with_arms"         default="false"/>
+  <!-- head pan/tilt (bus1, motor_id 7/8) is phase 3 too - not wired on the
+       robot yet. Without this, bus1's ros2_control component still gets
+       declared for head_pan/head_tilt alone and tries to open bus1_port,
+       which doesn't exist until the head is actually plugged in. -->
+  <xacro:arg name="with_head"         default="false"/>
   <xacro:property name="dims_file" value="$(find xlerobot_description)/config/robot_dimensions.yaml"/>
   <xacro:property name="dims" value="${xacro.load_yaml(dims_file)['xlerobot']}"/>
@@ -49,4 +54,5 @@
           use_mock_hardware="$(arg use_mock_hardware)"
           with_arms="$(arg with_arms)"
+          with_head="$(arg with_head)"
           dims="${dims}"/>
     </xacro:unless>

Commit message: Arm and head joints read-only by default (torque_off)
torque_off:=true declares the arm and head joints with state interfaces only, so
the driver leaves torque off and never writes to them. torque_off:=false restores
the position command interfaces.

File: src/xlerobot_description/urdf/xlerobot.ros2_control.xacro (robot description, xacro)
@@ -27,12 +27,16 @@
 -->
 <robot xmlns:xacro="http://www.ros.org/wiki/xacro">
-  <xacro:macro name="sts_position_joint" params="name id lower upper">
+  <!-- read_only: no command interface, so the driver disables torque on the joint and
+       never writes to it, while its state is still read every cycle. -->
+  <xacro:macro name="sts_position_joint" params="name id lower upper read_only:=false">
     <joint name="${name}">
       <param name="motor_id">${id}</param>
       <param name="operating_mode">0</param>
-      <command_interface name="position">
-        <param name="min">${lower}</param>
-        <param name="max">${upper}</param>
-      </command_interface>
+      <xacro:unless value="${read_only}">
+        <command_interface name="position">
+          <param name="min">${lower}</param>
+          <param name="max">${upper}</param>
+        </command_interface>
+      </xacro:unless>
       <state_interface name="position"/>
       <state_interface name="velocity"/>
@@ -46,13 +50,13 @@
   <!-- The six joints of one arm, IDs 1-6. Names and limits match so101_arm.xacro,
        which has the limits of the arm in upstream's URDF. -->
-  <xacro:macro name="sts_arm_joints" params="prefix">
-    <xacro:sts_position_joint name="${prefix}_shoulder_pan_joint"  id="1" lower="-2.16"      upper="2.16"/>
-    <xacro:sts_position_joint name="${prefix}_shoulder_lift_joint" id="2" lower="-0.22"      upper="3.37"/>
-    <xacro:sts_position_joint name="${prefix}_elbow_flex_joint"    id="3" lower="-0.22"      upper="3.14"/>
-    <xacro:sts_position_joint name="${prefix}_wrist_flex_joint"    id="4" lower="-1.6580628" upper="1.6580627"/>
-    <xacro:sts_position_joint name="${prefix}_wrist_roll_joint"    id="5" lower="-2.7438473" upper="2.8412063"/>
-    <xacro:sts_position_joint name="${prefix}_gripper_joint"       id="6" lower="-0.374533" upper="1.7453292"/>
+  <xacro:macro name="sts_arm_joints" params="prefix read_only">
+    <xacro:sts_position_joint name="${prefix}_shoulder_pan_joint"  id="1" lower="-2.16"      upper="2.16" read_only="${read_only}"/>
+    <xacro:sts_position_joint name="${prefix}_shoulder_lift_joint" id="2" lower="-0.22"      upper="3.37" read_only="${read_only}"/>
+    <xacro:sts_position_joint name="${prefix}_elbow_flex_joint"    id="3" lower="-0.22"      upper="3.14" read_only="${read_only}"/>
+    <xacro:sts_position_joint name="${prefix}_wrist_flex_joint"    id="4" lower="-1.6580628" upper="1.6580627" read_only="${read_only}"/>
+    <xacro:sts_position_joint name="${prefix}_wrist_roll_joint"    id="5" lower="-2.7438473" upper="2.8412063" read_only="${read_only}"/>
+    <xacro:sts_position_joint name="${prefix}_gripper_joint"       id="6" lower="-0.374533" upper="1.7453292" read_only="${read_only}"/>
   </xacro:macro>
-  <xacro:macro name="xlerobot_ros2_control" params="bus1_port bus2_port use_mock_hardware with_arms with_head dims">
+  <xacro:macro name="xlerobot_ros2_control" params="bus1_port bus2_port use_mock_hardware with_arms torque_off with_head dims">
     <xacro:property name="b"      value="${dims['base']}"/>
     <xacro:property name="h"      value="${dims['head']}"/>
@@ -73,11 +77,13 @@
         </hardware>
         <xacro:if value="${with_arms}">
-          <xacro:sts_arm_joints prefix="left_arm"/>
+          <xacro:sts_arm_joints prefix="left_arm" read_only="${torque_off}"/>
         </xacro:if>
         <xacro:if value="${with_head}">
           <xacro:sts_position_joint name="head_pan_joint"  id="7"
-                                    lower="${h['pan_limit_lower']}"  upper="${h['pan_limit_upper']}"/>
+                                    lower="${h['pan_limit_lower']}"  upper="${h['pan_limit_upper']}"
+                                    read_only="${torque_off}"/>
           <xacro:sts_position_joint name="head_tilt_joint" id="8"
-                                    lower="${h['tilt_limit_lower']}" upper="${h['tilt_limit_upper']}"/>
+                                    lower="${h['tilt_limit_lower']}" upper="${h['tilt_limit_upper']}"
+                                    read_only="${torque_off}"/>
         </xacro:if>
       </ros2_control>
@@ -92,5 +98,5 @@
       </hardware>
       <xacro:if value="${with_arms}">
-        <xacro:sts_arm_joints prefix="right_arm"/>
+        <xacro:sts_arm_joints prefix="right_arm" read_only="${torque_off}"/>
       </xacro:if>
       <!-- The RIGHT motor is mounted mirrored (confirmed on the real robot by

File: src/xlerobot_description/urdf/xlerobot.urdf.xacro (robot description, xacro)
@@ -28,4 +28,7 @@
   <!-- arms are phase 3, description only for now -->
   <xacro:arg name="with_arms"         default="false"/>
+  <!-- Arm and head joints without command interfaces: torque off, states only. Stays
+       true until they are calibrated, see docs/arms-bringup.md. Wheels are not affected. -->
+  <xacro:arg name="torque_off"    default="true"/>
   <!-- head pan/tilt (bus1, motor_id 7/8) is phase 3 too - not wired on the
        robot yet. Without this, bus1's ros2_control component still gets
@@ -72,4 +75,5 @@
           use_mock_hardware="$(arg use_mock_hardware)"
           with_arms="$(arg with_arms)"
+          torque_off="$(arg torque_off)"
           with_head="$(arg with_head)"
           dims="${dims}"/>

Commit message: Arm zero steps per arm, read off the arms held stretched straight

File: src/xlerobot_description/urdf/xlerobot.ros2_control.xacro (robot description, xacro)
@@ -53,18 +53,18 @@
        and match so101_arm.xacro: with direction +1 the model's joint is reversed against the
        source URDF, so the limits are mirrored. -->
-  <xacro:macro name="sts_arm_joint" params="name id j read_only">
+  <xacro:macro name="sts_arm_joint" params="name id j side read_only">
     <xacro:property name="m" value="${-j['direction']}"/>
     <xacro:sts_position_joint name="${name}" id="${id}"
         lower="${min(m * j['lower'], m * j['upper'])}" upper="${max(m * j['lower'], m * j['upper'])}"
-        center="${j['zero_step']}" read_only="${read_only}"/>
+        center="${j['zero_step'][side]}" read_only="${read_only}"/>
   </xacro:macro>
   <!-- The six joints of one arm, IDs 1-6, names as in so101_arm.xacro. -->
-  <xacro:macro name="sts_arm_joints" params="prefix read_only joints">
-    <xacro:sts_arm_joint name="${prefix}_shoulder_pan_joint"  id="1" j="${joints['shoulder_pan']}"  read_only="${read_only}"/>
-    <xacro:sts_arm_joint name="${prefix}_shoulder_lift_joint" id="2" j="${joints['shoulder_lift']}" read_only="${read_only}"/>
-    <xacro:sts_arm_joint name="${prefix}_elbow_flex_joint"    id="3" j="${joints['elbow_flex']}"    read_only="${read_only}"/>
-    <xacro:sts_arm_joint name="${prefix}_wrist_flex_joint"    id="4" j="${joints['wrist_flex']}"    read_only="${read_only}"/>
-    <xacro:sts_arm_joint name="${prefix}_wrist_roll_joint"    id="5" j="${joints['wrist_roll']}"    read_only="${read_only}"/>
-    <xacro:sts_arm_joint name="${prefix}_gripper_joint"       id="6" j="${joints['gripper']}"       read_only="${read_only}"/>
+  <xacro:macro name="sts_arm_joints" params="prefix side read_only joints">
+    <xacro:sts_arm_joint name="${prefix}_shoulder_pan_joint"  id="1" j="${joints['shoulder_pan']}" side="${side}"  read_only="${read_only}"/>
+    <xacro:sts_arm_joint name="${prefix}_shoulder_lift_joint" id="2" j="${joints['shoulder_lift']}" side="${side}" read_only="${read_only}"/>
+    <xacro:sts_arm_joint name="${prefix}_elbow_flex_joint"    id="3" j="${joints['elbow_flex']}" side="${side}"    read_only="${read_only}"/>
+    <xacro:sts_arm_joint name="${prefix}_wrist_flex_joint"    id="4" j="${joints['wrist_flex']}" side="${side}"    read_only="${read_only}"/>
+    <xacro:sts_arm_joint name="${prefix}_wrist_roll_joint"    id="5" j="${joints['wrist_roll']}" side="${side}"    read_only="${read_only}"/>
+    <xacro:sts_arm_joint name="${prefix}_gripper_joint"       id="6" j="${joints['gripper']}" side="${side}"       read_only="${read_only}"/>
   </xacro:macro>
   <xacro:macro name="xlerobot_ros2_control" params="bus1_port bus2_port use_mock_hardware with_arms torque_off with_head dims">
@@ -87,5 +87,5 @@
         </hardware>
         <xacro:if value="${with_arms}">
-          <xacro:sts_arm_joints prefix="left_arm" read_only="${torque_off}" joints="${dims['arms']['joints']}"/>
+          <xacro:sts_arm_joints prefix="left_arm" side="left" read_only="${torque_off}" joints="${dims['arms']['joints']}"/>
         </xacro:if>
         <xacro:if value="${with_head}">
@@ -112,5 +112,5 @@
       </hardware>
       <xacro:if value="${with_arms}">
-        <xacro:sts_arm_joints prefix="right_arm" read_only="${torque_off}" joints="${dims['arms']['joints']}"/>
+        <xacro:sts_arm_joints prefix="right_arm" side="right" read_only="${torque_off}" joints="${dims['arms']['joints']}"/>
       </xacro:if>
       <!-- The RIGHT motor is mounted mirrored (confirmed on the real robot by
