Commit message: Arm controllers, hold-on-activate, speed caps, e-stop tool, fake servo bus
joint_trajectory_controller per arm and gripper, spawned with with_arms torque_off:=false.
Driver-side limits and rate cap from robot_dimensions.yaml, tools/estop.py for every bus,
tools/fake_sts_bus.py to run the real driver without hardware.

File: src/xlerobot_description/urdf/so101_arm.xacro (robot description, xacro)
@@ -7,5 +7,5 @@
   stretched straight out to the side, and it folds by about +3 rad at the shoulder
   lift and elbow, which is how the real arms rest. Only the joint velocity limit
-  changed, the source has 0, 3 rad/s here so planners get a usable limit. Joint axes and
+  changed, the source has 0, arms.joints max_velocity here so planners get a usable limit. Joint axes and
   limits follow arms.joints in robot_dimensions.yaml: where the real servo goes the other
   way from the source's angle the axis is reversed and the limits mirrored.
@@ -281,5 +281,5 @@
       <origin xyz="0 -0.0452 0.0165" rpy="1.5708 0 0"/>
       <axis xyz="0 ${-1 * m_pan} 0"/>
-      <limit lower="${lo_pan}" upper="${hi_pan}" effort="3.35" velocity="3.0"/>
+      <limit lower="${lo_pan}" upper="${hi_pan}" effort="3.35" velocity="${joints['shoulder_pan']['max_velocity']}"/>
       <dynamics damping="0.6" friction="0.052"/>
     </joint>
@@ -289,5 +289,5 @@
       <origin xyz="0 0.1025 0.0306" rpy="1.5708 0 0"/>
       <axis xyz="${-1 * m_lift} 0 0"/>
-      <limit lower="${lo_lift}" upper="${hi_lift}" effort="3.35" velocity="3.0"/>
+      <limit lower="${lo_lift}" upper="${hi_lift}" effort="3.35" velocity="${joints['shoulder_lift']['max_velocity']}"/>
       <dynamics damping="0.6" friction="0.052"/>
     </joint>
@@ -297,5 +297,5 @@
       <origin xyz="0 0.11257 0.028" rpy="-1.5708 0 0"/>
       <axis xyz="${m_elbow} 0 0"/>
-      <limit lower="${lo_elbow}" upper="${hi_elbow}" effort="3.35" velocity="3.0"/>
+      <limit lower="${lo_elbow}" upper="${hi_elbow}" effort="3.35" velocity="${joints['elbow_flex']['max_velocity']}"/>
       <dynamics damping="0.6" friction="0.052"/>
     </joint>
@@ -305,5 +305,5 @@
       <origin xyz="0 0.0052 0.1349" rpy="-1.5708 0 0"/>
       <axis xyz="${m_wflex} 0 0"/>
-      <limit lower="${lo_wflex}" upper="${hi_wflex}" effort="3.35" velocity="3.0"/>
+      <limit lower="${lo_wflex}" upper="${hi_wflex}" effort="3.35" velocity="${joints['wrist_flex']['max_velocity']}"/>
       <dynamics damping="0.6" friction="0.052"/>
     </joint>
@@ -313,5 +313,5 @@
       <origin xyz="0 -0.0601 0" rpy="0 1.5707927 0"/>
       <axis xyz="0 ${-1 * m_roll} 0"/>
-      <limit lower="${lo_roll}" upper="${hi_roll}" effort="3.35" velocity="3.0"/>
+      <limit lower="${lo_roll}" upper="${hi_roll}" effort="3.35" velocity="${joints['wrist_roll']['max_velocity']}"/>
       <dynamics damping="0.6" friction="0.052"/>
     </joint>
@@ -321,5 +321,5 @@
       <origin xyz="-0.0202 -0.0244 0" rpy="3.1415854 -0.0000014 2.9531853"/>
       <axis xyz="0 0 ${m_grip}"/>
-      <limit lower="${lo_grip}" upper="${hi_grip}" effort="10" velocity="3.0"/>
+      <limit lower="${lo_grip}" upper="${hi_grip}" effort="10" velocity="${joints['gripper']['max_velocity']}"/>
       <dynamics damping="0.6" friction="0.052"/>
     </joint>

File: src/xlerobot_description/urdf/xlerobot.ros2_control.xacro (robot description, xacro)
@@ -29,5 +29,5 @@
   <!-- read_only: no command interface, so the driver disables torque on the joint and
        never writes to it, while its state is still read every cycle. -->
-  <xacro:macro name="sts_position_joint" params="name id lower upper center:=4095 read_only:=false">
+  <xacro:macro name="sts_position_joint" params="name id lower upper center:=4095 rate_limit:=0 read_only:=false">
     <joint name="${name}">
       <param name="motor_id">${id}</param>
@@ -35,4 +35,11 @@
       <!-- servo step that is 0 rad, the driver reports (center - step) -->
       <param name="position_center_steps">${center}</param>
+      <!-- the driver's own clamp, it ignores the command interface min/max below -->
+      <param name="min_position">${lower}</param>
+      <param name="max_position">${upper}</param>
+      <!-- cap on how fast the commanded position may move, rad/s, 0 = none. The driver holds
+           the target back to this speed, so a trajectory faster than that lags and the
+           controller aborts it. -->
+      <param name="position_rate_limit">${rate_limit}</param>
       <xacro:unless value="${read_only}">
         <command_interface name="position">
@@ -50,5 +57,6 @@
     </joint>
   </xacro:macro>
-  <!-- One arm joint. The limits and the centre come from arms.joints in robot_dimensions.yaml
+  <!-- One arm joint. The limits, the centre and the speed cap (1.25 x the planning velocity limit)
+       come from arms.joints in robot_dimensions.yaml
        and match so101_arm.xacro: with direction +1 the model's joint is reversed against the
        source URDF, so the limits are mirrored. -->
@@ -57,5 +65,5 @@
     <xacro:sts_position_joint name="${name}" id="${id}"
         lower="${min(m * j['lower'], m * j['upper'])}" upper="${max(m * j['lower'], m * j['upper'])}"
-        center="${j['zero_step'][side]}" read_only="${read_only}"/>
+        center="${j['zero_step'][side]}" rate_limit="${1.25 * j['max_velocity']}" read_only="${read_only}"/>
   </xacro:macro>
   <!-- The six joints of one arm, IDs 1-6, names as in so101_arm.xacro. -->
@@ -85,4 +93,5 @@
           <param name="baud_rate">1000000</param>
           <param name="enable_mock_mode">$(arg use_mock_hardware)</param>
+          <param name="proportional_vel_max">${dims['arms']['servo_speed_limit_steps']}</param>
         </hardware>
         <xacro:if value="${with_arms}">
@@ -110,4 +119,5 @@
         <param name="baud_rate">1000000</param>
         <param name="enable_mock_mode">$(arg use_mock_hardware)</param>
+        <param name="proportional_vel_max">${dims['arms']['servo_speed_limit_steps']}</param>
       </hardware>
       <xacro:if value="${with_arms}">

Commit message: Shared limit margin for the arm joints in the model and ros2_control
The trajectory controller shuts down when a joint is measured outside its URDF limits, and the
left elbow rests 2 degrees past the upstream limit at its hard stop.

File: src/xlerobot_description/urdf/so101_arm.xacro (robot description, xacro)
@@ -19,26 +19,26 @@
 -->
 <robot xmlns:xacro="http://www.ros.org/wiki/xacro">
-  <xacro:macro name="so101_arm" params="prefix parent xyz rpy joints wrist_camera:=true">
+  <xacro:macro name="so101_arm" params="prefix parent xyz rpy joints margin wrist_camera:=true">
     <!-- joint direction, see arms.joints in robot_dimensions.yaml: m is -1 to reverse the
          axis (and mirror the limits) where the servo step goes the same way as the joint
          angle. Reversing axis and angle together is the same pose. -->
     <xacro:property name="m_pan" value="${-joints['shoulder_pan']['direction']}"/>
-    <xacro:property name="lo_pan" value="${min(m_pan * joints['shoulder_pan']['lower'], m_pan * joints['shoulder_pan']['upper'])}"/>
-    <xacro:property name="hi_pan" value="${max(m_pan * joints['shoulder_pan']['lower'], m_pan * joints['shoulder_pan']['upper'])}"/>
+    <xacro:property name="lo_pan" value="${min(m_pan * joints['shoulder_pan']['lower'], m_pan * joints['shoulder_pan']['upper']) - margin}"/>
+    <xacro:property name="hi_pan" value="${max(m_pan * joints['shoulder_pan']['lower'], m_pan * joints['shoulder_pan']['upper']) + margin}"/>
     <xacro:property name="m_lift" value="${-joints['shoulder_lift']['direction']}"/>
-    <xacro:property name="lo_lift" value="${min(m_lift * joints['shoulder_lift']['lower'], m_lift * joints['shoulder_lift']['upper'])}"/>
-    <xacro:property name="hi_lift" value="${max(m_lift * joints['shoulder_lift']['lower'], m_lift * joints['shoulder_lift']['upper'])}"/>
+    <xacro:property name="lo_lift" value="${min(m_lift * joints['shoulder_lift']['lower'], m_lift * joints['shoulder_lift']['upper']) - margin}"/>
+    <xacro:property name="hi_lift" value="${max(m_lift * joints['shoulder_lift']['lower'], m_lift * joints['shoulder_lift']['upper']) + margin}"/>
     <xacro:property name="m_elbow" value="${-joints['elbow_flex']['direction']}"/>
-    <xacro:property name="lo_elbow" value="${min(m_elbow * joints['elbow_flex']['lower'], m_elbow * joints['elbow_flex']['upper'])}"/>
-    <xacro:property name="hi_elbow" value="${max(m_elbow * joints['elbow_flex']['lower'], m_elbow * joints['elbow_flex']['upper'])}"/>
+    <xacro:property name="lo_elbow" value="${min(m_elbow * joints['elbow_flex']['lower'], m_elbow * joints['elbow_flex']['upper']) - margin}"/>
+    <xacro:property name="hi_elbow" value="${max(m_elbow * joints['elbow_flex']['lower'], m_elbow * joints['elbow_flex']['upper']) + margin}"/>
     <xacro:property name="m_wflex" value="${-joints['wrist_flex']['direction']}"/>
-    <xacro:property name="lo_wflex" value="${min(m_wflex * joints['wrist_flex']['lower'], m_wflex * joints['wrist_flex']['upper'])}"/>
-    <xacro:property name="hi_wflex" value="${max(m_wflex * joints['wrist_flex']['lower'], m_wflex * joints['wrist_flex']['upper'])}"/>
+    <xacro:property name="lo_wflex" value="${min(m_wflex * joints['wrist_flex']['lower'], m_wflex * joints['wrist_flex']['upper']) - margin}"/>
+    <xacro:property name="hi_wflex" value="${max(m_wflex * joints['wrist_flex']['lower'], m_wflex * joints['wrist_flex']['upper']) + margin}"/>
     <xacro:property name="m_roll" value="${-joints['wrist_roll']['direction']}"/>
-    <xacro:property name="lo_roll" value="${min(m_roll * joints['wrist_roll']['lower'], m_roll * joints['wrist_roll']['upper'])}"/>
-    <xacro:property name="hi_roll" value="${max(m_roll * joints['wrist_roll']['lower'], m_roll * joints['wrist_roll']['upper'])}"/>
+    <xacro:property name="lo_roll" value="${min(m_roll * joints['wrist_roll']['lower'], m_roll * joints['wrist_roll']['upper']) - margin}"/>
+    <xacro:property name="hi_roll" value="${max(m_roll * joints['wrist_roll']['lower'], m_roll * joints['wrist_roll']['upper']) + margin}"/>
     <xacro:property name="m_grip" value="${-joints['gripper']['direction']}"/>
-    <xacro:property name="lo_grip" value="${min(m_grip * joints['gripper']['lower'], m_grip * joints['gripper']['upper'])}"/>
-    <xacro:property name="hi_grip" value="${max(m_grip * joints['gripper']['lower'], m_grip * joints['gripper']['upper'])}"/>
+    <xacro:property name="lo_grip" value="${min(m_grip * joints['gripper']['lower'], m_grip * joints['gripper']['upper']) - margin}"/>
+    <xacro:property name="hi_grip" value="${max(m_grip * joints['gripper']['lower'], m_grip * joints['gripper']['upper']) + margin}"/>
     <joint name="${prefix}_mount_joint" type="fixed">
       <parent link="${parent}"/>

File: src/xlerobot_description/urdf/xlerobot.ros2_control.xacro (robot description, xacro)
@@ -61,18 +61,18 @@
        and match so101_arm.xacro: with direction +1 the model's joint is reversed against the
        source URDF, so the limits are mirrored. -->
-  <xacro:macro name="sts_arm_joint" params="name id j side read_only">
+  <xacro:macro name="sts_arm_joint" params="name id j side margin read_only">
     <xacro:property name="m" value="${-j['direction']}"/>
     <xacro:sts_position_joint name="${name}" id="${id}"
-        lower="${min(m * j['lower'], m * j['upper'])}" upper="${max(m * j['lower'], m * j['upper'])}"
+        lower="${min(m * j['lower'], m * j['upper']) - margin}" upper="${max(m * j['lower'], m * j['upper']) + margin}"
         center="${j['zero_step'][side]}" rate_limit="${1.25 * j['max_velocity']}" read_only="${read_only}"/>
   </xacro:macro>
   <!-- The six joints of one arm, IDs 1-6, names as in so101_arm.xacro. -->
-  <xacro:macro name="sts_arm_joints" params="prefix side read_only joints">
-    <xacro:sts_arm_joint name="${prefix}_shoulder_pan_joint"  id="1" j="${joints['shoulder_pan']}" side="${side}"  read_only="${read_only}"/>
-    <xacro:sts_arm_joint name="${prefix}_shoulder_lift_joint" id="2" j="${joints['shoulder_lift']}" side="${side}" read_only="${read_only}"/>
-    <xacro:sts_arm_joint name="${prefix}_elbow_flex_joint"    id="3" j="${joints['elbow_flex']}" side="${side}"    read_only="${read_only}"/>
-    <xacro:sts_arm_joint name="${prefix}_wrist_flex_joint"    id="4" j="${joints['wrist_flex']}" side="${side}"    read_only="${read_only}"/>
-    <xacro:sts_arm_joint name="${prefix}_wrist_roll_joint"    id="5" j="${joints['wrist_roll']}" side="${side}"    read_only="${read_only}"/>
-    <xacro:sts_arm_joint name="${prefix}_gripper_joint"       id="6" j="${joints['gripper']}" side="${side}"       read_only="${read_only}"/>
+  <xacro:macro name="sts_arm_joints" params="prefix side read_only joints margin">
+    <xacro:sts_arm_joint name="${prefix}_shoulder_pan_joint"  id="1" j="${joints['shoulder_pan']}" side="${side}" margin="${margin}"  read_only="${read_only}"/>
+    <xacro:sts_arm_joint name="${prefix}_shoulder_lift_joint" id="2" j="${joints['shoulder_lift']}" side="${side}" margin="${margin}" read_only="${read_only}"/>
+    <xacro:sts_arm_joint name="${prefix}_elbow_flex_joint"    id="3" j="${joints['elbow_flex']}" side="${side}" margin="${margin}"    read_only="${read_only}"/>
+    <xacro:sts_arm_joint name="${prefix}_wrist_flex_joint"    id="4" j="${joints['wrist_flex']}" side="${side}" margin="${margin}"    read_only="${read_only}"/>
+    <xacro:sts_arm_joint name="${prefix}_wrist_roll_joint"    id="5" j="${joints['wrist_roll']}" side="${side}" margin="${margin}"    read_only="${read_only}"/>
+    <xacro:sts_arm_joint name="${prefix}_gripper_joint"       id="6" j="${joints['gripper']}" side="${side}" margin="${margin}"       read_only="${read_only}"/>
   </xacro:macro>
   <xacro:macro name="xlerobot_ros2_control" params="bus1_port bus2_port use_mock_hardware with_arms torque_off with_head dims">
@@ -96,5 +96,5 @@
         </hardware>
         <xacro:if value="${with_arms}">
-          <xacro:sts_arm_joints prefix="left_arm" side="left" read_only="${torque_off}" joints="${dims['arms']['joints']}"/>
+          <xacro:sts_arm_joints prefix="left_arm" side="left" read_only="${torque_off}" joints="${dims['arms']['joints']}" margin="${dims['arms']['limit_margin']}"/>
         </xacro:if>
         <xacro:if value="${with_head}">
@@ -122,5 +122,5 @@
       </hardware>
       <xacro:if value="${with_arms}">
-        <xacro:sts_arm_joints prefix="right_arm" side="right" read_only="${torque_off}" joints="${dims['arms']['joints']}"/>
+        <xacro:sts_arm_joints prefix="right_arm" side="right" read_only="${torque_off}" joints="${dims['arms']['joints']}" margin="${dims['arms']['limit_margin']}"/>
       </xacro:if>
       <!-- The RIGHT motor is mounted mirrored (confirmed on the real robot by

File: src/xlerobot_description/urdf/xlerobot.urdf.xacro (robot description, xacro)
@@ -60,8 +60,8 @@
     <xacro:property name="a" value="${dims['arms']}"/>
     <xacro:property name="pan_off" value="0.0452"/>
-    <xacro:so101_arm prefix="left_arm"  parent="body_link" joints="${a['joints']}"
+    <xacro:so101_arm prefix="left_arm"  parent="body_link" joints="${a['joints']}" margin="${a['limit_margin']}"
         xyz="${a['mount_x'] - pan_off * sin(a['left_yaw'])} ${-a['mount_y'] + pan_off * cos(a['left_yaw'])} ${a['mount_z']}"
         rpy="0 0 ${a['left_yaw']}"/>
-    <xacro:so101_arm prefix="right_arm" parent="body_link" joints="${a['joints']}"
+    <xacro:so101_arm prefix="right_arm" parent="body_link" joints="${a['joints']}" margin="${a['limit_margin']}"
         xyz="${a['mount_x'] - pan_off * sin(a['right_yaw'])}  ${a['mount_y'] + pan_off * cos(a['right_yaw'])} ${a['mount_z']}"
         rpy="0 0 ${a['right_yaw']}"/>
