Commit message: Description: real SO-101 arms, head on its mast, head camera frame
so101_arm.xacro was a stub of cylinders. It is now the SO-101 model from
so_arm_description (links, joints, inertials, limits), converted with a
prefix so both arms can be included, with meshes referenced from that
package. The only change is the joint velocity, 3 rad/s instead of the
source's 1e6, so planners get a usable limit. The wrist camera mount and
its optical frame come with it.

Arm mount pose is in robot_dimensions.yaml (arms: block), taken from
upstream XLeRobot's reference URDF, both arms facing forward. Not
measured on this robot. The head moves from the cart top to about 1.05 m
on a mast, also from upstream's numbers, with a placeholder mast rod so
it does not float.

New sensor value usbcam, now the default: the head camera the robot has
today, a webcam, with head_camera_link and head_camera_optical_frame.

ros2_control arm joints were named without the _joint suffix, so they
could never have matched the URDF or the sim's names. They now use
<prefix>_<joint>_joint and the SO-101 limits instead of placeholders.
bringup gets with_arms (default false), which also opens bus1.

File: src/xlerobot_description/urdf/head_pantilt.xacro (robot description, xacro)
@@ -8,4 +8,25 @@
   <xacro:macro name="xlerobot_head" params="dims parent">
     <xacro:property name="h" value="${dims['head']}"/>
+    <!-- Mast from the cart top plate up to the pan servo, a placeholder rod so the
+         head does not float. TODO swap for topbase1/2.stl. -->
+    <xacro:property name="mast_bottom" value="${dims['base']['body_height'] - 0.005}"/>
+    <xacro:property name="mast_length" value="${h['mount_z'] - 0.02 - mast_bottom}"/>
+    <link name="head_mast_link">
+      <visual>
+        <origin xyz="0 0 ${mast_length / 2.0}" rpy="0 0 0"/>
+        <geometry><cylinder radius="0.02" length="${mast_length}"/></geometry>
+        <material name="xle_accent"/>
+      </visual>
+      <inertial>
+        <origin xyz="0 0 ${mast_length / 2.0}" rpy="0 0 0"/>
+        <mass value="0.1"/>
+        <inertia ixx="1e-4" ixy="0" ixz="0" iyy="1e-4" iyz="0" izz="1e-5"/>
+      </inertial>
+    </link>
+    <joint name="head_mast_joint" type="fixed">
+      <parent link="${parent}"/>
+      <child  link="head_mast_link"/>
+      <origin xyz="${h['mount_x']} ${h['mount_y']} ${mast_bottom}" rpy="0 0 0"/>
+    </joint>
     <link name="head_pan_link">
       <visual>

File: src/xlerobot_description/urdf/sensors.xacro (robot description, xacro)
@@ -2,5 +2,5 @@
 <!--
   Sensor mount is sensor agnostic on purpose, see ADR-0003, the choice isn't
-  made yet. sensor arg picks one of: none, vlp16, gemini, realsense.
+  made yet. sensor arg picks one of: none, usbcam, vlp16, gemini, realsense.
   Head mount frame is head_camera_mount, from head_pantilt.xacro.
   Lidar mount point is a placeholder until we know where it actually goes,
@@ -9,4 +9,31 @@
 <robot xmlns:xacro="http://www.ros.org/wiki/xacro">
   <xacro:macro name="xlerobot_sensors" params="sensor dims">
+    <!-- The head camera the robot has today: a plain USB webcam, the same model
+         as the wrist cameras (bringup cameras:=true, config/cameras.yaml). Body
+         size and pose on the head are approximate, not measured. -->
+    <xacro:if value="${sensor == 'usbcam'}">
+      <link name="head_camera_link">
+        <visual>
+          <geometry><box size="0.02 0.05 0.03"/></geometry>
+          <material name="xle_black"/>
+        </visual>
+        <inertial>
+          <mass value="0.03"/>
+          <inertia ixx="1e-5" ixy="0" ixz="0" iyy="1e-5" iyz="0" izz="1e-5"/>
+        </inertial>
+      </link>
+      <joint name="head_camera_joint" type="fixed">
+        <parent link="head_camera_mount"/>
+        <child  link="head_camera_link"/>
+        <origin xyz="0 0 0" rpy="0 0 0"/>
+      </joint>
+      <!-- REP-103 optical frame, z forward -->
+      <link name="head_camera_optical_frame"/>
+      <joint name="head_camera_optical_joint" type="fixed">
+        <parent link="head_camera_link"/>
+        <child  link="head_camera_optical_frame"/>
+        <origin xyz="0 0 0" rpy="${-pi/2} 0 ${-pi/2}"/>
+      </joint>
+    </xacro:if>
     <xacro:if value="${sensor == 'realsense'}">
       <link name="head_camera_link">

File: src/xlerobot_description/urdf/so101_arm.xacro (robot description, xacro)
@@ -1,78 +1,443 @@
 <?xml version="1.0"?>
 <!--
-  Placeholder. Real SO-101 xacro is phase 3, joint limits and mesh
-  references pulled from adityakamath/so_arm_ros2 and cross-checked against
-  ros-physical-ai/ros2_so_arm, see ARCHITECTURE §3. This stub just gives
-  with_arms:=true something to attach so the toggle isn't broken.
-  6 joints per arm, matches IDs 1-6 on bus1 (left) / bus2 (right), see
-  ARCHITECTURE §1.1. Straight chain, no real geometry, no meshes.
+  SO-101 arm, one instance per arm, names prefixed (left_arm_shoulder_pan_joint,
+  left_arm_wrist_camera_optical_frame, ...).
+  Links, joints, inertials and joint limits are the SO-101 model from
+  adityakamath/so_arm_ros2's so_arm_description (Apache-2.0), converted with
+  a prefix so it can be included twice. Meshes are referenced from that
+  package, not copied. Only the joint velocity changed: the source has 1e6
+  (it leaves the cap to the servo firmware), 3 rad/s here so planners get a
+  usable limit.
+  The wrist camera mount and frames are the SO-101 wrist camera design, its
+  optical frame follows REP-103 (z forward). Not measured on this robot.
+  parent/xyz/rpy place the arm's base_link. wrist_camera:=false leaves out the
+  camera links.
 -->
 <robot xmlns:xacro="http://www.ros.org/wiki/xacro">
-  <xacro:macro name="so101_arm" params="prefix parent xyz rpy">
-    <link name="${prefix}_mount"/>
+  <xacro:macro name="so101_arm" params="prefix parent xyz rpy wrist_camera:=true">
+    <material name="${prefix}_light_grey">
+      <color rgba="0.8 0.8 0.8 1.0"/>
+    </material>
+    <material name="${prefix}_charcoal">
+      <color rgba="0.15 0.15 0.15 1.0"/>
+    </material>
     <joint name="${prefix}_mount_joint" type="fixed">
       <parent link="${parent}"/>
-      <child  link="${prefix}_mount"/>
+      <child link="${prefix}_base_link"/>
       <origin xyz="${xyz}" rpy="${rpy}"/>
     </joint>
-    <xacro:macro name="stub_link" params="name">
-      <link name="${name}">
-        <visual>
-          <geometry><cylinder radius="0.02" length="0.08"/></geometry>
-          <material name="xle_accent"/>
-        </visual>
+    <link name="${prefix}_base_link">
+      <inertial>
+        <origin rpy="0 0 0" xyz="0.0137179 -5.19711e-05 0.0334843"/>
+        <mass value="0.147"/>
+        <inertia ixx="0.000114686" ixy="-4.59787e-07" ixz="4.97151e-06" iyy="0.000136117" iyz="9.75275e-08" izz="0.000130364"/>
+      </inertial>
+      <visual>
+        <origin rpy="1.5708 -1.67685e-15 1.5708" xyz="-0.00636471 -9.94414e-05 -0.0024"/>
+        <geometry>
+          <mesh filename="package://so_arm_description/meshes/so101/base_motor_holder_so101_v1.stl"/>
+        </geometry>
+        <material name="${prefix}_light_grey"/>
+      </visual>
+      <collision>
+        <origin rpy="1.5708 -1.67685e-15 1.5708" xyz="-0.00636471 -9.94414e-05 -0.0024"/>
+        <geometry>
+          <mesh filename="package://so_arm_description/meshes/so101/base_motor_holder_so101_v1.stl"/>
+        </geometry>
+      </collision>
+      <visual>
+        <origin rpy="1.5708 -2.78073e-29 1.5708" xyz="-0.00636471 -8.97657e-09 -0.0024"/>
+        <geometry>
+          <mesh filename="package://so_arm_description/meshes/so101/base_so101_v2.stl"/>
+        </geometry>
+        <material name="${prefix}_light_grey"/>
+      </visual>
+      <collision>
+        <origin rpy="1.5708 -2.78073e-29 1.5708" xyz="-0.00636471 -8.97657e-09 -0.0024"/>
+        <geometry>
+          <mesh filename="package://so_arm_description/meshes/so101/base_so101_v2.stl"/>
+        </geometry>
+      </collision>
+      <visual>
+        <origin rpy="-8.21148e-16 7.84513e-18 1.249e-15" xyz="0.0263353 -8.97657e-09 0.0437"/>
+        <geometry>
+          <mesh filename="package://so_arm_description/meshes/so101/sts3215_03a_v1.stl"/>
+        </geometry>
+        <material name="${prefix}_charcoal"/>
+      </visual>
+      <collision>
+        <origin rpy="-8.21148e-16 7.84513e-18 1.249e-15" xyz="0.0263353 -8.97657e-09 0.0437"/>
+        <geometry>
+          <mesh filename="package://so_arm_description/meshes/so101/sts3215_03a_v1.stl"/>
+        </geometry>
+      </collision>
+      <visual>
+        <origin rpy="1.5708 -1.35493e-14 1.5708" xyz="-0.0309827 -0.000199441 0.0474"/>
+        <geometry>
+          <mesh filename="package://so_arm_description/meshes/so101/waveshare_mounting_plate_so101_v2.stl"/>
+        </geometry>
+        <material name="${prefix}_light_grey"/>
+      </visual>
+      <collision>
+        <origin rpy="1.5708 -1.35493e-14 1.5708" xyz="-0.0309827 -0.000199441 0.0474"/>
+        <geometry>
+          <mesh filename="package://so_arm_description/meshes/so101/waveshare_mounting_plate_so101_v2.stl"/>
+        </geometry>
+      </collision>
+    </link>
+    <link name="${prefix}_shoulder_link">
+      <inertial>
+        <origin rpy="0 0 0" xyz="0.0307604 -1.66727e-05 0.0252713"/>
+        <mass value="0.100006"/>
+        <inertia ixx="8.3759e-05" ixy="-7.55525e-08" ixz="-1.16342e-06" iyy="8.10403e-05" iyz="-1.54663e-07" izz="2.39783e-05"/>
+      </inertial>
+      <visual>
+        <origin rpy="1.5708 -1.5708 0" xyz="0.0303992 0.000422241 0.0417"/>
+        <geometry>
+          <mesh filename="package://so_arm_description/meshes/so101/sts3215_03a_v1.stl"/>
+        </geometry>
+        <material name="${prefix}_charcoal"/>
+      </visual>
+      <collision>
+        <origin rpy="1.5708 -1.5708 0" xyz="0.0303992 0.000422241 0.0417"/>
+        <geometry>
+          <mesh filename="package://so_arm_description/meshes/so101/sts3215_03a_v1.stl"/>
+        </geometry>
+      </collision>
+      <visual>
+        <origin rpy="1.5708 1.5708 0" xyz="0.0675992 -0.000177759 -0.0158499"/>
+        <geometry>
+          <mesh filename="package://so_arm_description/meshes/so101/motor_holder_so101_base_v1.stl"/>
+        </geometry>
+        <material name="${prefix}_light_grey"/>
+      </visual>
+      <collision>
+        <origin rpy="1.5708 1.5708 0" xyz="0.0675992 -0.000177759 -0.0158499"/>
+        <geometry>
+          <mesh filename="package://so_arm_description/meshes/so101/motor_holder_so101_base_v1.stl"/>
+        </geometry>
+      </collision>
+      <visual>
+        <origin rpy="1.5708 0 3.14159" xyz="-0.0122008 2.22413e-05 -0.0464"/>
+        <geometry>
+          <mesh filename="package://so_arm_description/meshes/so101/rotation_pitch_so101_v1.stl"/>
+        </geometry>
+        <material name="${prefix}_light_grey"/>
+      </visual>
+      <collision>
+        <origin rpy="1.5708 0 3.14159" xyz="-0.0122008 2.22413e-05 -0.0464"/>
+        <geometry>
+          <mesh filename="package://so_arm_description/meshes/so101/rotation_pitch_so101_v1.stl"/>
+        </geometry>
+      </collision>
+    </link>
+    <link name="${prefix}_upper_arm_link">
+      <inertial>
+        <origin rpy="0 0 0" xyz="-0.0898471 -0.00838224 0.0184089"/>
+        <mass value="0.103"/>
+        <inertia ixx="4.08002e-05" ixy="-1.97819e-05" ixz="-4.03016e-08" iyy="0.000147318" iyz="8.97326e-09" izz="0.000142487"/>
+      </inertial>
+      <visual>
+        <origin rpy="-3.14159 -5.27356e-16 -1.5708" xyz="-0.11257 -0.0155 0.0187"/>
+        <geometry>
+          <mesh filename="package://so_arm_description/meshes/so101/sts3215_03a_v1.stl"/>
+        </geometry>
+        <material name="${prefix}_charcoal"/>
+      </visual>
+      <collision>
+        <origin rpy="-3.14159 -5.27356e-16 -1.5708" xyz="-0.11257 -0.0155 0.0187"/>
+        <geometry>
+          <mesh filename="package://so_arm_description/meshes/so101/sts3215_03a_v1.stl"/>
+        </geometry>
+      </collision>
+      <visual>
+        <origin rpy="3.14159 -0 -1.30911e-30" xyz="-0.065085 0.012 0.0182"/>
+        <geometry>
+          <mesh filename="package://so_arm_description/meshes/so101/upper_arm_so101_v1.stl"/>
+        </geometry>
+        <material name="${prefix}_light_grey"/>
+      </visual>
+      <collision>
+        <origin rpy="3.14159 -0 -1.30911e-30" xyz="-0.065085 0.012 0.0182"/>
+        <geometry>
+          <mesh filename="package://so_arm_description/meshes/so101/upper_arm_so101_v1.stl"/>
+        </geometry>
+      </collision>
+    </link>
+    <link name="${prefix}_lower_arm_link">
+      <inertial>
+        <origin rpy="0 0 0" xyz="-0.0980701 0.00324376 0.0182831"/>
+        <mass value="0.104"/>
+        <inertia ixx="2.87438e-05" ixy="7.41152e-06" ixz="1.26409e-06" iyy="0.000159844" iyz="-4.90188e-08" izz="0.00014529"/>
+      </inertial>
+      <visual>
+        <origin rpy="3.14159 -0 6.67202e-31" xyz="-0.0648499 -0.032 0.0182"/>
+        <geometry>
+          <mesh filename="package://so_arm_description/meshes/so101/under_arm_so101_v1.stl"/>
+        </geometry>
+        <material name="${prefix}_light_grey"/>
+      </visual>
+      <collision>
+        <origin rpy="3.14159 -0 6.67202e-31" xyz="-0.0648499 -0.032 0.0182"/>
+        <geometry>
+          <mesh filename="package://so_arm_description/meshes/so101/under_arm_so101_v1.stl"/>
+        </geometry>
+      </collision>
+      <visual>
+        <origin rpy="-3.14159 -2.55351e-15 -1.83387e-30" xyz="-0.0648499 -0.032 0.018"/>
+        <geometry>
+          <mesh filename="package://so_arm_description/meshes/so101/motor_holder_so101_wrist_v1.stl"/>
+        </geometry>
+        <material name="${prefix}_light_grey"/>
+      </visual>
+      <collision>
+        <origin rpy="-3.14159 -2.55351e-15 -1.83387e-30" xyz="-0.0648499 -0.032 0.018"/>
+        <geometry>
+          <mesh filename="package://so_arm_description/meshes/so101/motor_holder_so101_wrist_v1.stl"/>
+        </geometry>
+      </collision>
+      <visual>
+        <origin rpy="-3.14159 -7.88861e-31 -3.14159" xyz="-0.1224 0.0052 0.0187"/>
+        <geometry>
+          <mesh filename="package://so_arm_description/meshes/so101/sts3215_03a_v1.stl"/>
+        </geometry>
+        <material name="${prefix}_charcoal"/>
+      </visual>
+      <collision>
+        <origin rpy="-3.14159 -7.88861e-31 -3.14159" xyz="-0.1224 0.0052 0.0187"/>
+        <geometry>
+          <mesh filename="package://so_arm_description/meshes/so101/sts3215_03a_v1.stl"/>
+        </geometry>
+      </collision>
+    </link>
+    <link name="${prefix}_wrist_link">
+      <inertial>
+        <origin rpy="0 0 0" xyz="-0.000103312 -0.0386143 0.0281156"/>
+        <mass value="0.079"/>
+        <inertia ixx="3.68263e-05" ixy="1.7893e-08" ixz="-5.28128e-08" iyy="2.5391e-05" iyz="3.6412e-06" izz="2.1e-05"/>
+      </inertial>
+      <visual>
+        <origin rpy="1.5708 1.5708 0" xyz="8.32667e-17 -0.0424 0.0306"/>
+        <geometry>
+          <mesh filename="package://so_arm_description/meshes/so101/sts3215_03a_no_horn_v1.stl"/>
+        </geometry>
+        <material name="${prefix}_charcoal"/>
+      </visual>
+      <collision>
+        <origin rpy="1.5708 1.5708 0" xyz="8.32667e-17 -0.0424 0.0306"/>
+        <geometry>
+          <mesh filename="package://so_arm_description/meshes/so101/sts3215_03a_no_horn_v1.stl"/>
+        </geometry>
+      </collision>
+      <visual>
+        <origin rpy="-1.5708 -1.5708 0" xyz="0 -0.028 0.0181"/>
+        <geometry>
+          <mesh filename="package://so_arm_description/meshes/so101/wrist_roll_pitch_so101_v2.stl"/>
+        </geometry>
+        <material name="${prefix}_light_grey"/>
+      </visual>
+      <collision>
+        <origin rpy="-1.5708 -1.5708 0" xyz="0 -0.028 0.0181"/>
+        <geometry>
+          <mesh filename="package://so_arm_description/meshes/so101/wrist_roll_pitch_so101_v2.stl"/>
+        </geometry>
+      </collision>
+    </link>
+    <link name="${prefix}_gripper_link">
+      <inertial>
+        <origin rpy="0 0 0" xyz="0.000213627 0.000245138 -0.025187"/>
+        <mass value="0.087"/>
+        <inertia ixx="2.75087e-05" ixy="-3.35241e-07" ixz="-5.7352e-06" iyy="4.33657e-05" iyz="-5.17847e-08" izz="3.45059e-05"/>
+      </inertial>
+      <visual>
+        <origin rpy="-1.5708 -5.19179e-17 -1.66533e-16" xyz="0.0077 0.0001 -0.0234"/>
+        <geometry>
+          <mesh filename="package://so_arm_description/meshes/so101/sts3215_03a_v1.stl"/>
+        </geometry>
+        <material name="${prefix}_charcoal"/>
+      </visual>
+      <collision>
+        <origin rpy="-1.5708 -5.19179e-17 -1.66533e-16" xyz="0.0077 0.0001 -0.0234"/>
+        <geometry>
+          <mesh filename="package://so_arm_description/meshes/so101/sts3215_03a_v1.stl"/>
+        </geometry>
+      </collision>
+      <visual>
+        <origin rpy="-3.14159 -5.55112e-17 0" xyz="8.32667e-17 -0.000218214 0.000949706"/>
+        <geometry>
+          <mesh filename="package://so_arm_description/meshes/so101/wrist_roll_follower_so101_v1.stl"/>
+        </geometry>
+        <material name="${prefix}_light_grey"/>
+      </visual>
+      <collision>
+        <origin rpy="-3.14159 -5.55112e-17 0" xyz="8.32667e-17 -0.000218214 0.000949706"/>
+        <geometry>
+          <mesh filename="package://so_arm_description/meshes/so101/wrist_roll_follower_so101_v1.stl"/>
+        </geometry>
+      </collision>
+    </link>
+    <link name="${prefix}_end_effector_link">
+      <inertial>
+        <origin rpy="0 0 0" xyz="0 0 0"/>
+        <mass value="1e-9"/>
+        <inertia ixx="0" ixy="0" ixz="0" iyy="0" iyz="0" izz="0"/>
+      </inertial>
+    </link>
+    <xacro:if value="${wrist_camera}">
+      <link name="${prefix}_wrist_camera_mount_link">
         <inertial>
-          <mass value="0.05"/>
+          <origin rpy="0 0 0" xyz="0 0 0"/>
+          <mass value="0.02"/>
           <inertia ixx="1e-5" ixy="0" ixz="0" iyy="1e-5" iyz="0" izz="1e-5"/>
         </inertial>
+        <visual>
+          <origin rpy="0 0 0" xyz="0 0 0"/>
+          <geometry>
+            <mesh filename="package://so_arm_description/meshes/so101/wrist_camera_mount_so101_v1.stl" scale="0.001 0.001 0.001"/>
+          </geometry>
+          <material name="${prefix}_light_grey"/>
+        </visual>
+        <collision>
+          <origin rpy="0 0 0" xyz="0 0 0"/>
+          <geometry>
+            <mesh filename="package://so_arm_description/meshes/so101/wrist_camera_mount_so101_v1.stl" scale="0.001 0.001 0.001"/>
+          </geometry>
+        </collision>
       </link>
-    </xacro:macro>
-    <xacro:stub_link name="${prefix}_shoulder_pan_link"/>
-    <xacro:stub_link name="${prefix}_shoulder_lift_link"/>
-    <xacro:stub_link name="${prefix}_elbow_flex_link"/>
-    <xacro:stub_link name="${prefix}_wrist_flex_link"/>
-    <xacro:stub_link name="${prefix}_wrist_roll_link"/>
-    <xacro:stub_link name="${prefix}_gripper_link"/>
+    </xacro:if>
+    <xacro:if value="${wrist_camera}">
+      <link name="${prefix}_wrist_camera_body_link">
+        <inertial>
+          <origin rpy="0 0 0" xyz="0 0 0"/>
+          <mass value="0.015"/>
+          <inertia ixx="1e-5" ixy="0" ixz="0" iyy="1e-5" iyz="0" izz="1e-5"/>
+        </inertial>
+        <visual>
+          <origin rpy="0 0 0" xyz="0 0 0"/>
+          <geometry>
+            <mesh filename="package://so_arm_description/meshes/so101/wrist_camera_so101_v1.stl"/>
+          </geometry>
+          <material name="${prefix}_charcoal"/>
+        </visual>
+        <collision>
+          <origin rpy="0 0 0" xyz="0 0 0"/>
+          <geometry>
+            <mesh filename="package://so_arm_description/meshes/so101/wrist_camera_so101_v1.stl"/>
+          </geometry>
+        </collision>
+      </link>
+    </xacro:if>
+    <xacro:if value="${wrist_camera}">
+      <link name="${prefix}_wrist_camera_frame">
+        <inertial>
+          <origin rpy="0 0 0" xyz="0 0 0"/>
+          <mass value="1e-9"/>
+          <inertia ixx="0" ixy="0" ixz="0" iyy="0" iyz="0" izz="0"/>
+        </inertial>
+      </link>
+    </xacro:if>
+    <xacro:if value="${wrist_camera}">
+      <link name="${prefix}_wrist_camera_optical_frame">
+        <inertial>
+          <origin rpy="0 0 0" xyz="0 0 0"/>
+          <mass value="1e-9"/>
+          <inertia ixx="0" ixy="0" ixz="0" iyy="0" iyz="0" izz="0"/>
+        </inertial>
+      </link>
+    </xacro:if>
+    <link name="${prefix}_moving_jaw_link">
+      <inertial>
+        <origin rpy="0 0 0" xyz="-0.00157495 -0.0300244 0.0192755"/>
+        <mass value="0.012"/>
+        <inertia ixx="6.61427e-06" ixy="-3.19807e-07" ixz="-5.90717e-09" iyy="1.89032e-06" iyz="-1.09945e-07" izz="5.28738e-06"/>
+      </inertial>
+      <visual>
+        <origin rpy="9.53145e-17 6.93889e-18 1.24077e-24" xyz="-5.55112e-17 -5.55112e-17 0.0189"/>
+        <geometry>
+          <mesh filename="package://so_arm_description/meshes/so101/moving_jaw_so101_v1.stl"/>
+        </geometry>
+        <material name="${prefix}_light_grey"/>
+      </visual>
+      <collision>
+        <origin rpy="9.53145e-17 6.93889e-18 1.24077e-24" xyz="-5.55112e-17 -5.55112e-17 0.0189"/>
+        <geometry>
+          <mesh filename="package://so_arm_description/meshes/so101/moving_jaw_so101_v1.stl"/>
+        </geometry>
+      </collision>
+    </link>
     <joint name="${prefix}_shoulder_pan_joint" type="revolute">
-      <parent link="${prefix}_mount"/>
-      <child link="${prefix}_shoulder_pan_link"/>
-      <origin xyz="0 0 0" rpy="0 0 0"/>
+      <parent link="${prefix}_base_link"/>
+      <child link="${prefix}_shoulder_link"/>
+      <origin xyz="0.0388353 -8.97657e-09 0.0624"/>
       <axis xyz="0 0 1"/>
-      <limit lower="-3.14" upper="3.14" effort="5" velocity="3"/>
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