Commit message: Description: real SO-101 arms, head on its mast, head camera frame
so101_arm.xacro was a stub of cylinders. It is now the SO-101 model from
so_arm_description (links, joints, inertials, limits), converted with a
prefix so both arms can be included, with meshes referenced from that
package. The only change is the joint velocity, 3 rad/s instead of the
source's 1e6, so planners get a usable limit. The wrist camera mount and
its optical frame come with it.

Arm mount pose is in robot_dimensions.yaml (arms: block), taken from
upstream XLeRobot's reference URDF, both arms facing forward. Not
measured on this robot. The head moves from the cart top to about 1.05 m
on a mast, also from upstream's numbers, with a placeholder mast rod so
it does not float.

New sensor value usbcam, now the default: the head camera the robot has
today, a webcam, with head_camera_link and head_camera_optical_frame.

ros2_control arm joints were named without the _joint suffix, so they
could never have matched the URDF or the sim's names. They now use
<prefix>_<joint>_joint and the SO-101 limits instead of placeholders.
bringup gets with_arms (default false), which also opens bus1.

File: src/xlerobot_description/urdf/xlerobot.ros2_control.xacro (robot description, xacro)
@@ -44,4 +44,14 @@
     </joint>
   </xacro:macro>
+  <!-- The six SO-101 joints of one arm, IDs 1-6. Names match so101_arm.xacro,
+       limits are the SO-101 model's (so_arm_description). -->
+  <xacro:macro name="sts_arm_joints" params="prefix">
+    <xacro:sts_position_joint name="${prefix}_shoulder_pan_joint"  id="1" lower="-1.91986" upper="1.91986"/>
+    <xacro:sts_position_joint name="${prefix}_shoulder_lift_joint" id="2" lower="-1.74533" upper="1.74533"/>
+    <xacro:sts_position_joint name="${prefix}_elbow_flex_joint"    id="3" lower="-1.69"    upper="1.69"/>
+    <xacro:sts_position_joint name="${prefix}_wrist_flex_joint"    id="4" lower="-1.65806" upper="1.65806"/>
+    <xacro:sts_position_joint name="${prefix}_wrist_roll_joint"    id="5" lower="-2.74385" upper="2.84121"/>
+    <xacro:sts_position_joint name="${prefix}_gripper_joint"       id="6" lower="-1.74533" upper="0.174533"/>
+  </xacro:macro>
   <xacro:macro name="xlerobot_ros2_control" params="bus1_port bus2_port use_mock_hardware with_arms with_head dims">
     <xacro:property name="b"      value="${dims['base']}"/>
@@ -63,12 +73,5 @@
         </hardware>
         <xacro:if value="${with_arms}">
-          <!-- phase 3. Limits are placeholders, check against
-               adityakamath/so_arm_ros2 and ros-physical-ai/ros2_so_arm -->
-          <xacro:sts_position_joint name="left_arm_shoulder_pan"   id="1" lower="-3.14" upper="3.14"/>
-          <xacro:sts_position_joint name="left_arm_shoulder_lift"  id="2" lower="-1.75" upper="1.75"/>
-          <xacro:sts_position_joint name="left_arm_elbow_flex"     id="3" lower="-1.75" upper="1.75"/>
-          <xacro:sts_position_joint name="left_arm_wrist_flex"     id="4" lower="-1.75" upper="1.75"/>
-          <xacro:sts_position_joint name="left_arm_wrist_roll"     id="5" lower="-3.14" upper="3.14"/>
-          <xacro:sts_position_joint name="left_arm_gripper"        id="6" lower="0.0"   upper="1.75"/>
+          <xacro:sts_arm_joints prefix="left_arm"/>
         </xacro:if>
         <xacro:if value="${with_head}">
@@ -89,10 +92,5 @@
       </hardware>
       <xacro:if value="${with_arms}">
-        <xacro:sts_position_joint name="right_arm_shoulder_pan"  id="1" lower="-3.14" upper="3.14"/>
-        <xacro:sts_position_joint name="right_arm_shoulder_lift" id="2" lower="-1.75" upper="1.75"/>
-        <xacro:sts_position_joint name="right_arm_elbow_flex"    id="3" lower="-1.75" upper="1.75"/>
-        <xacro:sts_position_joint name="right_arm_wrist_flex"    id="4" lower="-1.75" upper="1.75"/>
-        <xacro:sts_position_joint name="right_arm_wrist_roll"    id="5" lower="-3.14" upper="3.14"/>
-        <xacro:sts_position_joint name="right_arm_gripper"       id="6" lower="0.0"   upper="1.75"/>
+        <xacro:sts_arm_joints prefix="right_arm"/>
       </xacro:if>
       <!-- The RIGHT motor is mounted mirrored (confirmed on the real robot by

File: src/xlerobot_description/urdf/xlerobot.urdf.xacro (robot description, xacro)
@@ -21,6 +21,7 @@
   <xacro:arg name="bus1_port"         default="/dev/xle-bus1"/>
   <xacro:arg name="bus2_port"         default="/dev/xle-bus2"/>
-  <!-- none | vlp16 | gemini | realsense, see ADR-0003 -->
-  <xacro:arg name="sensor"            default="none"/>
+  <!-- none | usbcam | vlp16 | gemini | realsense, see ADR-0003. usbcam is the head
+       camera the robot has today. -->
+  <xacro:arg name="sensor"            default="usbcam"/>
   <!-- arms are phase 3, description only for now -->
   <xacro:arg name="with_arms"         default="false"/>
@@ -41,8 +42,11 @@
   <xacro:if value="$(arg with_arms)">
     <xacro:include filename="$(find xlerobot_description)/urdf/so101_arm.xacro"/>
-    <!-- TODO mount offsets not measured. 0.4.0 top base allows different arm
-         directions, so this is a build choice, not a constant. -->
-    <xacro:so101_arm prefix="left_arm"  parent="base_link" xyz="0  0.12 0.78" rpy="0 0 0"/>
-    <xacro:so101_arm prefix="right_arm" parent="base_link" xyz="0 -0.12 0.78" rpy="0 0 0"/>
+    <!-- Mount pose from robot_dimensions.yaml, not measured yet. 0.4.0 top base
+         allows different arm directions, so the yaw is a build choice. -->
+    <xacro:property name="a" value="${dims['arms']}"/>
+    <xacro:so101_arm prefix="left_arm"  parent="base_link"
+        xyz="${a['mount_x']}  ${a['mount_y']} ${a['mount_z']}" rpy="0 0 ${a['mount_yaw']}"/>
+    <xacro:so101_arm prefix="right_arm" parent="base_link"
+        xyz="${a['mount_x']} ${-a['mount_y']} ${a['mount_z']}" rpy="0 0 ${a['mount_yaw']}"/>
   </xacro:if>
   <xacro:if value="$(arg use_ros2_control)">

Commit message: Description: arms, neck and head from the shared XLeRobot URDF
The arms, neck and head were built from other parts (generic SO-101 meshes,
a placeholder rod), which did not look like the robot. They are now the ones
in simulation/xlerobot/xlerobot.urdf of the XLeRobot repo: same meshes
(copied to meshes/upstream, 4 MB), link frames, joint origins and axes,
inertials and limits, converted by script with our joint and frame names.
The zero pose is that URDF's, the arms stretched out to the side, and the
shoulder lift and elbow fold by about +3 rad, which is how the real arms rest.

Positions: the mast axis is 70 mm from the rim of the top basket nearest the
drive wheels (measured), x=0.056. The arm pan axes are at the mast's x and
273 mm apart (CAD, confirmed on the robot), that URDF has them 310 mm apart.
The base origin follows each arm's yaw so the axis stays put. Each arm's yaw is
its own setting (right_yaw, left_yaw), default the original URDF's, since the
0.4.0 arm base can be mounted in any direction.

Heights, and the cart's position relative to the drive axle, are still that
URDF's, not measured. ros2_control arm and head limits follow the URDF's, the
so_arm_description dependency is gone.

File: src/xlerobot_description/urdf/head_pantilt.xacro (robot description, xacro)
@@ -1,67 +1,99 @@
 <?xml version="1.0"?>
 <!--
-  Head pan/tilt, IDs 7 and 8 on bus1. Frame names kept the same as upstream so
-  code written against their URDF still works.
-  TODO swap the boxes for topbase1/2.stl and tophead3/4.stl.
+  Neck and head pan/tilt, IDs 7 and 8 on bus1.
+  Converted from simulation/xlerobot/xlerobot.urdf of the XLeRobot repo
+  (xlerobot_urdf.zip): the printed top base, neck and head meshes
+  (meshes/upstream), link frames, joint origins and axes. The pan axis position
+  in base_link comes from robot_dimensions.yaml (head: mount_x/y/z), the top base
+  and everything above it follows from that. The head tilt link is turned 180
+  degrees about z, as in upstream, so its x axis points backwards; the camera
+  mount frame accounts for that. Pan/tilt limits are upstream's, TODO check them
+  against the mechanical stops.
 -->
 <robot xmlns:xacro="http://www.ros.org/wiki/xacro">
   <xacro:macro name="xlerobot_head" params="dims parent">
     <xacro:property name="h" value="${dims['head']}"/>
-    <!-- Mast from the cart top plate up to the pan servo, a placeholder rod so the
-         head does not float. TODO swap for topbase1/2.stl. -->
-    <xacro:property name="mast_bottom" value="${dims['base']['body_height'] - 0.005}"/>
-    <xacro:property name="mast_length" value="${h['mount_z'] - 0.02 - mast_bottom}"/>
-    <link name="head_mast_link">
+    <!-- top base sits 0.323 m below and 0.103 m ahead of the pan axis -->
+    <joint name="top_base_joint" type="fixed">
+      <parent link="${parent}"/>
+      <child link="top_base_link"/>
+      <origin xyz="${h['mount_x'] + 0.103} ${h['mount_y']} ${h['mount_z'] - 0.323}" rpy="0 0 0"/>
+    </joint>
+    <link name="top_base_link">
+      <inertial>
+        <origin xyz="0 0 0" rpy="0 0 0"/>
+        <mass value="0.2542"/>
+        <inertia ixx="0.0045" ixy="0" ixz="0" iyy="0.005" iyz="0" izz="0.0045"/>
+      </inertial>
       <visual>
-        <origin xyz="0 0 ${mast_length / 2.0}" rpy="0 0 0"/>
-        <geometry><cylinder radius="0.02" length="${mast_length}"/></geometry>
-        <material name="xle_accent"/>
+        <origin xyz="-0.44 -0.005 -0.6" rpy="0 0 0"/>
+        <geometry>
+          <mesh filename="package://xlerobot_description/meshes/upstream/topbase1.stl" scale="0.001 0.001 0.001"/>
+        </geometry>
+        <material name="xle_part"/>
       </visual>
+      <visual>
+        <origin xyz="-0.298 0.006 -0.715" rpy="0 0 3.14"/>
+        <geometry>
+          <mesh filename="package://xlerobot_description/meshes/upstream/topbase2.stl" scale="0.001 0.001 0.001"/>
+        </geometry>
+        <material name="xle_motor"/>
+      </visual>
+    </link>
+    <link name="head_pan_link">
       <inertial>
-        <origin xyz="0 0 ${mast_length / 2.0}" rpy="0 0 0"/>
-        <mass value="0.1"/>
-        <inertia ixx="1e-4" ixy="0" ixz="0" iyy="1e-4" iyz="0" izz="1e-5"/>
+        <origin xyz="0 0 0" rpy="0 0 0"/>
+        <mass value="0.2556"/>
+        <inertia ixx="0.0129" ixy="0" ixz="0" iyy="0.0095" iyz="0" izz="0.0184"/>
       </inertial>
-    </link>
-    <joint name="head_mast_joint" type="fixed">
-      <parent link="${parent}"/>
-      <child  link="head_mast_link"/>
-      <origin xyz="${h['mount_x']} ${h['mount_y']} ${mast_bottom}" rpy="0 0 0"/>
-    </joint>
-    <link name="head_pan_link">
       <visual>
-        <geometry><cylinder radius="0.035" length="0.04"/></geometry>
-        <material name="xle_accent"/>
+        <origin xyz="-0.335 -0.005 -0.923" rpy="0 0 0"/>
+        <geometry>
+          <mesh filename="package://xlerobot_description/meshes/upstream/tophead1.stl" scale="0.001 0.001 0.001"/>
+        </geometry>
+        <material name="xle_part"/>
       </visual>
-      <inertial>
-        <mass value="0.1"/>
-        <inertia ixx="1e-4" ixy="0" ixz="0" iyy="1e-4" iyz="0" izz="1e-4"/>
-      </inertial>
+      <visual>
+        <origin xyz="1.17 -0.009 0.262" rpy="-3.141592 -1.57 -3.141592"/>
+        <geometry>
+          <mesh filename="package://xlerobot_description/meshes/upstream/tophead4.stl" scale="0.001 0.001 0.001"/>
+        </geometry>
+        <material name="xle_motor"/>
+      </visual>
     </link>
     <joint name="head_pan_joint" type="revolute">
-      <parent link="${parent}"/>
-      <child  link="head_pan_link"/>
-      <origin xyz="${h['mount_x']} ${h['mount_y']} ${h['mount_z']}" rpy="0 0 0"/>
+      <parent link="top_base_link"/>
+      <child link="head_pan_link"/>
+      <origin xyz="-0.103 0 0.323" rpy="0 0 0"/>
       <axis xyz="0 0 1"/>
-      <limit lower="${h['pan_limit_lower']}" upper="${h['pan_limit_upper']}"
-             effort="2.0" velocity="3.0"/>
+      <limit lower="${h['pan_limit_lower']}" upper="${h['pan_limit_upper']}" effort="2.0" velocity="3.0"/>
     </joint>
     <link name="head_tilt_link">
+      <inertial>
+        <origin xyz="0 0 0" rpy="0 0 0"/>
+        <mass value="0.02087"/>
+        <inertia ixx="0.0061" ixy="0" ixz="0" iyy="0.0014" iyz="0" izz="0.0061"/>
+      </inertial>
       <visual>
-        <geometry><box size="0.06 0.09 0.04"/></geometry>
-        <material name="xle_accent"/>
+        <origin xyz="0.16265 -0.006 -1.16815" rpy="0 0 0"/>
+        <geometry>
+          <mesh filename="package://xlerobot_description/meshes/upstream/tophead5.stl" scale="0.001 0.001 0.001"/>
+        </geometry>
+        <material name="xle_part"/>
       </visual>
-      <inertial>
-        <mass value="0.1"/>
-        <inertia ixx="1e-4" ixy="0" ixz="0" iyy="1e-4" iyz="0" izz="1e-4"/>
-      </inertial>
+      <visual>
+        <origin xyz="0.16265 -0.006 -1.16815" rpy="0 0 0"/>
+        <geometry>
+          <mesh filename="package://xlerobot_description/meshes/upstream/tophead6.stl" scale="0.001 0.001 0.001"/>
+        </geometry>
+        <material name="xle_motor"/>
+      </visual>
     </link>
     <joint name="head_tilt_joint" type="revolute">
       <parent link="head_pan_link"/>
-      <child  link="head_tilt_link"/>
-      <origin xyz="0 0 0.04" rpy="0 0 0"/>
+      <child link="head_tilt_link"/>
+      <origin xyz="0.001 0.002 0.09815" rpy="0 0 3.1415927"/>
       <axis xyz="0 1 0"/>
-      <limit lower="${h['tilt_limit_lower']}" upper="${h['tilt_limit_upper']}"
-             effort="2.0" velocity="3.0"/>
+      <limit lower="${h['tilt_limit_lower']}" upper="${h['tilt_limit_upper']}" effort="2.0" velocity="3.0"/>
     </joint>
     <!-- sensor gets attached here, in sensors.xacro -->
@@ -69,6 +101,6 @@
     <joint name="head_camera_mount_joint" type="fixed">
       <parent link="head_tilt_link"/>
-      <child  link="head_camera_mount"/>
-      <origin xyz="0.03 0 0" rpy="0 0 0"/>
+      <child link="head_camera_mount"/>
+      <origin xyz="0.025 0 0.03" rpy="0 0 0"/>
     </joint>
   </xacro:macro>

File: src/xlerobot_description/urdf/materials.xacro (robot description, xacro)
@@ -5,3 +5,6 @@
   <material name="xle_accent"><color rgba="0.20 0.45 0.75 1.0"/></material>
   <material name="xle_white"> <color rgba="0.85 0.85 0.85 1.0"/></material>
+  <!-- printed parts and servos of the arms, neck and head, as in upstream's URDF -->
+  <material name="xle_part">  <color rgba="0.30 0.30 0.30 1.0"/></material>
+  <material name="xle_motor"> <color rgba="0.10 0.10 0.10 1.0"/></material>
 </robot>
