Commit message: Description: arms, neck and head from the shared XLeRobot URDF
The arms, neck and head were built from other parts (generic SO-101 meshes,
a placeholder rod), which did not look like the robot. They are now the ones
in simulation/xlerobot/xlerobot.urdf of the XLeRobot repo: same meshes
(copied to meshes/upstream, 4 MB), link frames, joint origins and axes,
inertials and limits, converted by script with our joint and frame names.
The zero pose is that URDF's, the arms stretched out to the side, and the
shoulder lift and elbow fold by about +3 rad, which is how the real arms rest.

Positions: the mast axis is 70 mm from the rim of the top basket nearest the
drive wheels (measured), x=0.056. The arm pan axes are at the mast's x and
273 mm apart (CAD, confirmed on the robot), that URDF has them 310 mm apart.
The base origin follows each arm's yaw so the axis stays put. Each arm's yaw is
its own setting (right_yaw, left_yaw), default the original URDF's, since the
0.4.0 arm base can be mounted in any direction.

Heights, and the cart's position relative to the drive axle, are still that
URDF's, not measured. ros2_control arm and head limits follow the URDF's, the
so_arm_description dependency is gone.

File: src/xlerobot_description/urdf/so101_arm.xacro (robot description, xacro)
@@ -1,25 +1,21 @@
 <?xml version="1.0"?>
 <!--
-  SO-101 arm, one instance per arm, names prefixed (left_arm_shoulder_pan_joint,
-  left_arm_wrist_camera_optical_frame, ...).
-  Links, joints, inertials and joint limits are the SO-101 model from
-  adityakamath/so_arm_ros2's so_arm_description (Apache-2.0), converted with
-  a prefix so it can be included twice. Meshes are referenced from that
-  package, not copied. Only the joint velocity changed: the source has 1e6
-  (it leaves the cap to the servo firmware), 3 rad/s here so planners get a
-  usable limit.
-  The wrist camera mount and frames are the SO-101 wrist camera design, its
-  optical frame follows REP-103 (z forward). Not measured on this robot.
-  parent/xyz/rpy place the arm's base_link. wrist_camera:=false leaves out the
-  camera links.
+  One arm, names prefixed (left_arm_shoulder_pan_joint, left_arm_wrist_camera_optical_frame, ...).
+  Converted from the arm in simulation/xlerobot/xlerobot.urdf of the XLeRobot
+  repo (xlerobot_urdf.zip): same meshes (meshes/upstream), link frames, joint
+  origins, axes, limits and inertials. The zero pose is that URDF's, the arm
+  stretched straight out to the side, and it folds by about +3 rad at the shoulder
+  lift and elbow, which is how the real arms rest. Only the joint velocity limit
+  changed, the source has 0, 3 rad/s here so planners get a usable limit.
+  Frame names follow the ros2_control joints and the sim, not upstream's
+  (upstream calls the arm on the right side *_L). The wrist camera is upstream's
+  Right/Left_Arm_Camera, its optical frame is REP-103 (z forward, the camera looks
+  along the fixed jaw).
+  parent/xyz/rpy place the arm's base_link. upstream mounts the arm on the right
+  side (y<0) with rpy 0 and the one on the left (y>0) turned 180 degrees about z.
+  wrist_camera:=false leaves out the camera links.
 -->
 <robot xmlns:xacro="http://www.ros.org/wiki/xacro">
   <xacro:macro name="so101_arm" params="prefix parent xyz rpy wrist_camera:=true">
-    <material name="${prefix}_light_grey">
-      <color rgba="0.8 0.8 0.8 1.0"/>
-    </material>
-    <material name="${prefix}_charcoal">
-      <color rgba="0.15 0.15 0.15 1.0"/>
-    </material>
     <joint name="${prefix}_mount_joint" type="fixed">
       <parent link="${parent}"/>
@@ -29,58 +25,32 @@
     <link name="${prefix}_base_link">
       <inertial>
-        <origin rpy="0 0 0" xyz="0.0137179 -5.19711e-05 0.0334843"/>
+        <origin xyz="0.0137179 -0.000052 0.0334843" rpy="0 0 0"/>
         <mass value="0.147"/>
-        <inertia ixx="0.000114686" ixy="-4.59787e-07" ixz="4.97151e-06" iyy="0.000136117" iyz="9.75275e-08" izz="0.000130364"/>
-      </inertial>
-      <visual>
-        <origin rpy="1.5708 -1.67685e-15 1.5708" xyz="-0.00636471 -9.94414e-05 -0.0024"/>
-        <geometry>
-          <mesh filename="package://so_arm_description/meshes/so101/base_motor_holder_so101_v1.stl"/>
-        </geometry>
-        <material name="${prefix}_light_grey"/>
-      </visual>
-      <collision>
-        <origin rpy="1.5708 -1.67685e-15 1.5708" xyz="-0.00636471 -9.94414e-05 -0.0024"/>
-        <geometry>
-          <mesh filename="package://so_arm_description/meshes/so101/base_motor_holder_so101_v1.stl"/>
-        </geometry>
-      </collision>
-      <visual>
-        <origin rpy="1.5708 -2.78073e-29 1.5708" xyz="-0.00636471 -8.97657e-09 -0.0024"/>
-        <geometry>
-          <mesh filename="package://so_arm_description/meshes/so101/base_so101_v2.stl"/>
-        </geometry>
-        <material name="${prefix}_light_grey"/>
-      </visual>
-      <collision>
-        <origin rpy="1.5708 -2.78073e-29 1.5708" xyz="-0.00636471 -8.97657e-09 -0.0024"/>
-        <geometry>
-          <mesh filename="package://so_arm_description/meshes/so101/base_so101_v2.stl"/>
-        </geometry>
-      </collision>
-      <visual>
-        <origin rpy="-8.21148e-16 7.84513e-18 1.249e-15" xyz="0.0263353 -8.97657e-09 0.0437"/>
-        <geometry>
-          <mesh filename="package://so_arm_description/meshes/so101/sts3215_03a_v1.stl"/>
-        </geometry>
-        <material name="${prefix}_charcoal"/>
-      </visual>
-      <collision>
-        <origin rpy="-8.21148e-16 7.84513e-18 1.249e-15" xyz="0.0263353 -8.97657e-09 0.0437"/>
-        <geometry>
-          <mesh filename="package://so_arm_description/meshes/so101/sts3215_03a_v1.stl"/>
-        </geometry>
-      </collision>
-      <visual>
-        <origin rpy="1.5708 -1.35493e-14 1.5708" xyz="-0.0309827 -0.000199441 0.0474"/>
-        <geometry>
-          <mesh filename="package://so_arm_description/meshes/so101/waveshare_mounting_plate_so101_v2.stl"/>
-        </geometry>
-        <material name="${prefix}_light_grey"/>
-      </visual>
-      <collision>
-        <origin rpy="1.5708 -1.35493e-14 1.5708" xyz="-0.0309827 -0.000199441 0.0474"/>
-        <geometry>
-          <mesh filename="package://so_arm_description/meshes/so101/waveshare_mounting_plate_so101_v2.stl"/>
+        <inertia ixx="0.0001147" ixy="-0.0000005" ixz="0.000005" iyy="0.0001361" iyz="0.0000001" izz="0.0001304"/>
+      </inertial>
+      <visual>
+        <origin xyz="0 0 0" rpy="0 0 0"/>
+        <geometry>
+          <mesh filename="package://xlerobot_description/meshes/upstream/Base.stl"/>
+        </geometry>
+        <material name="xle_part"/>
+      </visual>
+      <collision>
+        <origin xyz="0 0 0" rpy="0 0 0"/>
+        <geometry>
+          <mesh filename="package://xlerobot_description/meshes/upstream/Base.stl"/>
+        </geometry>
+      </collision>
+      <visual>
+        <origin xyz="0 0 0" rpy="0 0 0"/>
+        <geometry>
+          <mesh filename="package://xlerobot_description/meshes/upstream/Base_Motor.stl"/>
+        </geometry>
+        <material name="xle_motor"/>
+      </visual>
+      <collision>
+        <origin xyz="0 0 0" rpy="0 0 0"/>
+        <geometry>
+          <mesh filename="package://xlerobot_description/meshes/upstream/Base_Motor.stl"/>
         </geometry>
       </collision>
@@ -88,45 +58,32 @@
     <link name="${prefix}_shoulder_link">
       <inertial>
-        <origin rpy="0 0 0" xyz="0.0307604 -1.66727e-05 0.0252713"/>
+        <origin xyz="-0.0307604 -0.0000167 -0.0252713" rpy="0 0 0"/>
         <mass value="0.100006"/>
-        <inertia ixx="8.3759e-05" ixy="-7.55525e-08" ixz="-1.16342e-06" iyy="8.10403e-05" iyz="-1.54663e-07" izz="2.39783e-05"/>
-      </inertial>
-      <visual>
-        <origin rpy="1.5708 -1.5708 0" xyz="0.0303992 0.000422241 0.0417"/>
-        <geometry>
-          <mesh filename="package://so_arm_description/meshes/so101/sts3215_03a_v1.stl"/>
-        </geometry>
-        <material name="${prefix}_charcoal"/>
-      </visual>
-      <collision>
-        <origin rpy="1.5708 -1.5708 0" xyz="0.0303992 0.000422241 0.0417"/>
-        <geometry>
-          <mesh filename="package://so_arm_description/meshes/so101/sts3215_03a_v1.stl"/>
-        </geometry>
-      </collision>
-      <visual>
-        <origin rpy="1.5708 1.5708 0" xyz="0.0675992 -0.000177759 -0.0158499"/>
-        <geometry>
-          <mesh filename="package://so_arm_description/meshes/so101/motor_holder_so101_base_v1.stl"/>
-        </geometry>
-        <material name="${prefix}_light_grey"/>
-      </visual>
-      <collision>
-        <origin rpy="1.5708 1.5708 0" xyz="0.0675992 -0.000177759 -0.0158499"/>
-        <geometry>
-          <mesh filename="package://so_arm_description/meshes/so101/motor_holder_so101_base_v1.stl"/>
-        </geometry>
-      </collision>
-      <visual>
-        <origin rpy="1.5708 0 3.14159" xyz="-0.0122008 2.22413e-05 -0.0464"/>
-        <geometry>
-          <mesh filename="package://so_arm_description/meshes/so101/rotation_pitch_so101_v1.stl"/>
-        </geometry>
-        <material name="${prefix}_light_grey"/>
-      </visual>
-      <collision>
-        <origin rpy="1.5708 0 3.14159" xyz="-0.0122008 2.22413e-05 -0.0464"/>
-        <geometry>
-          <mesh filename="package://so_arm_description/meshes/so101/rotation_pitch_so101_v1.stl"/>
+        <inertia ixx="0.0000838" ixy="0.0000001" ixz="-0.0000012" iyy="0.000081" iyz="0.0000002" izz="0.000024"/>
+      </inertial>
+      <visual>
+        <origin xyz="0 0 0" rpy="0 0 0"/>
+        <geometry>
+          <mesh filename="package://xlerobot_description/meshes/upstream/Rotation_Pitch.stl"/>
+        </geometry>
+        <material name="xle_part"/>
+      </visual>
+      <collision>
+        <origin xyz="0 0 0" rpy="0 0 0"/>
+        <geometry>
+          <mesh filename="package://xlerobot_description/meshes/upstream/Rotation_Pitch.stl"/>
+        </geometry>
+      </collision>
+      <visual>
+        <origin xyz="0 0 0" rpy="0 0 0"/>
+        <geometry>
+          <mesh filename="package://xlerobot_description/meshes/upstream/Rotation_Pitch_Motor.stl"/>
+        </geometry>
+        <material name="xle_motor"/>
+      </visual>
+      <collision>
+        <origin xyz="0 0 0" rpy="0 0 0"/>
+        <geometry>
+          <mesh filename="package://xlerobot_description/meshes/upstream/Rotation_Pitch_Motor.stl"/>
         </geometry>
       </collision>
@@ -134,32 +91,32 @@
     <link name="${prefix}_upper_arm_link">
       <inertial>
-        <origin rpy="0 0 0" xyz="-0.0898471 -0.00838224 0.0184089"/>
+        <origin xyz="-0.0898471 -0.0083822 0.0184089" rpy="0 0 0"/>
         <mass value="0.103"/>
-        <inertia ixx="4.08002e-05" ixy="-1.97819e-05" ixz="-4.03016e-08" iyy="0.000147318" iyz="8.97326e-09" izz="0.000142487"/>
-      </inertial>
-      <visual>
-        <origin rpy="-3.14159 -5.27356e-16 -1.5708" xyz="-0.11257 -0.0155 0.0187"/>
-        <geometry>
-          <mesh filename="package://so_arm_description/meshes/so101/sts3215_03a_v1.stl"/>
-        </geometry>
-        <material name="${prefix}_charcoal"/>
-      </visual>
-      <collision>
-        <origin rpy="-3.14159 -5.27356e-16 -1.5708" xyz="-0.11257 -0.0155 0.0187"/>
-        <geometry>
-          <mesh filename="package://so_arm_description/meshes/so101/sts3215_03a_v1.stl"/>
-        </geometry>
-      </collision>
-      <visual>
-        <origin rpy="3.14159 -0 -1.30911e-30" xyz="-0.065085 0.012 0.0182"/>
-        <geometry>
-          <mesh filename="package://so_arm_description/meshes/so101/upper_arm_so101_v1.stl"/>
-        </geometry>
-        <material name="${prefix}_light_grey"/>
-      </visual>
-      <collision>
-        <origin rpy="3.14159 -0 -1.30911e-30" xyz="-0.065085 0.012 0.0182"/>
-        <geometry>
-          <mesh filename="package://so_arm_description/meshes/so101/upper_arm_so101_v1.stl"/>
+        <inertia ixx="0.0000408" ixy="-0.0000198" ixz="0" iyy="0.0001473" iyz="0" izz="0.0001425"/>
+      </inertial>
+      <visual>
+        <origin xyz="0 0 0" rpy="0 0 0"/>
+        <geometry>
+          <mesh filename="package://xlerobot_description/meshes/upstream/Upper_Arm.stl"/>
+        </geometry>
+        <material name="xle_part"/>
+      </visual>
+      <collision>
+        <origin xyz="0 0 0" rpy="0 0 0"/>
+        <geometry>
+          <mesh filename="package://xlerobot_description/meshes/upstream/Upper_Arm.stl"/>
+        </geometry>
+      </collision>
+      <visual>
+        <origin xyz="0 0 0" rpy="0 0 0"/>
+        <geometry>
+          <mesh filename="package://xlerobot_description/meshes/upstream/Upper_Arm_Motor.stl"/>
+        </geometry>
+        <material name="xle_motor"/>
+      </visual>
+      <collision>
+        <origin xyz="0 0 0" rpy="0 0 0"/>
+        <geometry>
+          <mesh filename="package://xlerobot_description/meshes/upstream/Upper_Arm_Motor.stl"/>
         </geometry>
       </collision>
@@ -167,45 +124,32 @@
     <link name="${prefix}_lower_arm_link">
       <inertial>
-        <origin rpy="0 0 0" xyz="-0.0980701 0.00324376 0.0182831"/>
+        <origin xyz="-0.0980701 0.0032438 0.0182831" rpy="0 0 0"/>
         <mass value="0.104"/>
-        <inertia ixx="2.87438e-05" ixy="7.41152e-06" ixz="1.26409e-06" iyy="0.000159844" iyz="-4.90188e-08" izz="0.00014529"/>
-      </inertial>
-      <visual>
-        <origin rpy="3.14159 -0 6.67202e-31" xyz="-0.0648499 -0.032 0.0182"/>
-        <geometry>
-          <mesh filename="package://so_arm_description/meshes/so101/under_arm_so101_v1.stl"/>
-        </geometry>
-        <material name="${prefix}_light_grey"/>
-      </visual>
-      <collision>
-        <origin rpy="3.14159 -0 6.67202e-31" xyz="-0.0648499 -0.032 0.0182"/>
-        <geometry>
-          <mesh filename="package://so_arm_description/meshes/so101/under_arm_so101_v1.stl"/>
-        </geometry>
-      </collision>
-      <visual>
-        <origin rpy="-3.14159 -2.55351e-15 -1.83387e-30" xyz="-0.0648499 -0.032 0.018"/>
-        <geometry>
-          <mesh filename="package://so_arm_description/meshes/so101/motor_holder_so101_wrist_v1.stl"/>
-        </geometry>
-        <material name="${prefix}_light_grey"/>
-      </visual>
-      <collision>
-        <origin rpy="-3.14159 -2.55351e-15 -1.83387e-30" xyz="-0.0648499 -0.032 0.018"/>
-        <geometry>
-          <mesh filename="package://so_arm_description/meshes/so101/motor_holder_so101_wrist_v1.stl"/>
-        </geometry>
-      </collision>
-      <visual>
-        <origin rpy="-3.14159 -7.88861e-31 -3.14159" xyz="-0.1224 0.0052 0.0187"/>
-        <geometry>
-          <mesh filename="package://so_arm_description/meshes/so101/sts3215_03a_v1.stl"/>
-        </geometry>
-        <material name="${prefix}_charcoal"/>
-      </visual>
-      <collision>
-        <origin rpy="-3.14159 -7.88861e-31 -3.14159" xyz="-0.1224 0.0052 0.0187"/>
-        <geometry>
-          <mesh filename="package://so_arm_description/meshes/so101/sts3215_03a_v1.stl"/>
+        <inertia ixx="0.0000287" ixy="0.0000074" ixz="0.0000013" iyy="0.0001598" iyz="0" izz="0.0001453"/>
+      </inertial>
+      <visual>
+        <origin xyz="0 0 0" rpy="0 0 0"/>
+        <geometry>
+          <mesh filename="package://xlerobot_description/meshes/upstream/Lower_Arm.stl"/>
+        </geometry>
+        <material name="xle_part"/>
+      </visual>
+      <collision>
+        <origin xyz="0 0 0" rpy="0 0 0"/>
+        <geometry>
+          <mesh filename="package://xlerobot_description/meshes/upstream/Lower_Arm.stl"/>
+        </geometry>
+      </collision>
+      <visual>
+        <origin xyz="0 0 0" rpy="0 0 0"/>
+        <geometry>
+          <mesh filename="package://xlerobot_description/meshes/upstream/Lower_Arm_Motor.stl"/>
+        </geometry>
+        <material name="xle_motor"/>
+      </visual>
+      <collision>
+        <origin xyz="0 0 0" rpy="0 0 0"/>
+        <geometry>
+          <mesh filename="package://xlerobot_description/meshes/upstream/Lower_Arm_Motor.stl"/>
         </geometry>
       </collision>
@@ -213,32 +157,32 @@
     <link name="${prefix}_wrist_link">
       <inertial>
-        <origin rpy="0 0 0" xyz="-0.000103312 -0.0386143 0.0281156"/>
+        <origin xyz="-0.0001033 -0.0386143 0.0281156" rpy="0 0 0"/>
         <mass value="0.079"/>
-        <inertia ixx="3.68263e-05" ixy="1.7893e-08" ixz="-5.28128e-08" iyy="2.5391e-05" iyz="3.6412e-06" izz="2.1e-05"/>
-      </inertial>
-      <visual>
-        <origin rpy="1.5708 1.5708 0" xyz="8.32667e-17 -0.0424 0.0306"/>
-        <geometry>
-          <mesh filename="package://so_arm_description/meshes/so101/sts3215_03a_no_horn_v1.stl"/>
-        </geometry>
-        <material name="${prefix}_charcoal"/>
-      </visual>
-      <collision>
-        <origin rpy="1.5708 1.5708 0" xyz="8.32667e-17 -0.0424 0.0306"/>
-        <geometry>
-          <mesh filename="package://so_arm_description/meshes/so101/sts3215_03a_no_horn_v1.stl"/>
-        </geometry>
-      </collision>
-      <visual>
-        <origin rpy="-1.5708 -1.5708 0" xyz="0 -0.028 0.0181"/>
-        <geometry>
-          <mesh filename="package://so_arm_description/meshes/so101/wrist_roll_pitch_so101_v2.stl"/>
-        </geometry>
-        <material name="${prefix}_light_grey"/>
-      </visual>
-      <collision>
-        <origin rpy="-1.5708 -1.5708 0" xyz="0 -0.028 0.0181"/>
-        <geometry>
-          <mesh filename="package://so_arm_description/meshes/so101/wrist_roll_pitch_so101_v2.stl"/>
+        <inertia ixx="0.0000368" ixy="0" ixz="-0.0000001" iyy="0.0000254" iyz="0.0000036" izz="0.000021"/>
+      </inertial>
+      <visual>
+        <origin xyz="0 0 0" rpy="0 0 0"/>
+        <geometry>
+          <mesh filename="package://xlerobot_description/meshes/upstream/Wrist_Pitch_Roll.stl"/>
+        </geometry>
+        <material name="xle_part"/>
+      </visual>
+      <collision>
+        <origin xyz="0 0 0" rpy="0 0 0"/>
+        <geometry>
+          <mesh filename="package://xlerobot_description/meshes/upstream/Wrist_Pitch_Roll.stl"/>
+        </geometry>
+      </collision>
+      <visual>
+        <origin xyz="0 0 0" rpy="0 0 0"/>
+        <geometry>
+          <mesh filename="package://xlerobot_description/meshes/upstream/Wrist_Pitch_Roll_Motor.stl"/>
+        </geometry>
+        <material name="xle_motor"/>
+      </visual>
+      <collision>
+        <origin xyz="0 0 0" rpy="0 0 0"/>
+        <geometry>
+          <mesh filename="package://xlerobot_description/meshes/upstream/Wrist_Pitch_Roll_Motor.stl"/>
         </geometry>
       </collision>
@@ -246,121 +190,64 @@
     <link name="${prefix}_gripper_link">
       <inertial>
-        <origin rpy="0 0 0" xyz="0.000213627 0.000245138 -0.025187"/>
+        <origin xyz="0.0002136 0.0002451 -0.025187" rpy="0 0 0"/>
         <mass value="0.087"/>
-        <inertia ixx="2.75087e-05" ixy="-3.35241e-07" ixz="-5.7352e-06" iyy="4.33657e-05" iyz="-5.17847e-08" izz="3.45059e-05"/>
-      </inertial>
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
File: src/xlerobot_description/urdf/xlerobot.ros2_control.xacro (robot description, xacro)
@@ -44,13 +44,13 @@
     </joint>
   </xacro:macro>
-  <!-- The six SO-101 joints of one arm, IDs 1-6. Names match so101_arm.xacro,
-       limits are the SO-101 model's (so_arm_description). -->
+  <!-- The six joints of one arm, IDs 1-6. Names and limits match so101_arm.xacro,
+       which has the limits of the arm in upstream's URDF. -->
   <xacro:macro name="sts_arm_joints" params="prefix">
-    <xacro:sts_position_joint name="${prefix}_shoulder_pan_joint"  id="1" lower="-1.91986" upper="1.91986"/>
-    <xacro:sts_position_joint name="${prefix}_shoulder_lift_joint" id="2" lower="-1.74533" upper="1.74533"/>
-    <xacro:sts_position_joint name="${prefix}_elbow_flex_joint"    id="3" lower="-1.69"    upper="1.69"/>
-    <xacro:sts_position_joint name="${prefix}_wrist_flex_joint"    id="4" lower="-1.65806" upper="1.65806"/>
-    <xacro:sts_position_joint name="${prefix}_wrist_roll_joint"    id="5" lower="-2.74385" upper="2.84121"/>
-    <xacro:sts_position_joint name="${prefix}_gripper_joint"       id="6" lower="-1.74533" upper="0.174533"/>
+    <xacro:sts_position_joint name="${prefix}_shoulder_pan_joint"  id="1" lower="-2.16"      upper="2.16"/>
+    <xacro:sts_position_joint name="${prefix}_shoulder_lift_joint" id="2" lower="-0.22"      upper="3.37"/>
+    <xacro:sts_position_joint name="${prefix}_elbow_flex_joint"    id="3" lower="-0.22"      upper="3.14"/>
+    <xacro:sts_position_joint name="${prefix}_wrist_flex_joint"    id="4" lower="-1.6580628" upper="1.6580627"/>
+    <xacro:sts_position_joint name="${prefix}_wrist_roll_joint"    id="5" lower="-2.7438473" upper="2.8412063"/>
+    <xacro:sts_position_joint name="${prefix}_gripper_joint"       id="6" lower="-0.374533" upper="1.7453292"/>
   </xacro:macro>
   <xacro:macro name="xlerobot_ros2_control" params="bus1_port bus2_port use_mock_hardware with_arms with_head dims">

File: src/xlerobot_description/urdf/xlerobot.urdf.xacro (robot description, xacro)
@@ -42,11 +42,19 @@
   <xacro:if value="$(arg with_arms)">
     <xacro:include filename="$(find xlerobot_description)/urdf/so101_arm.xacro"/>
-    <!-- Mount pose from robot_dimensions.yaml, not measured yet. 0.4.0 top base
-         allows different arm directions, so the yaw is a build choice. -->
+    <!-- Mount pose from robot_dimensions.yaml: where each shoulder pan axis is
+         (mount_x, +-mount_y) and each arm's yaw (left_yaw, right_yaw). The pan axis
+         is 0.0452 m to the side of the arm's base_link in the base's own frame, so
+         the base origin moves with the yaw to keep the axis where it is. Upstream
+         mounts the right arm (y<0) with yaw 0 and the left one turned 180 degrees,
+         both stretch out sideways at zero. The 0.4.0 top base allows other
+         directions, so the yaws are a build choice. -->
     <xacro:property name="a" value="${dims['arms']}"/>
+    <xacro:property name="pan_off" value="0.0452"/>
     <xacro:so101_arm prefix="left_arm"  parent="base_link"
-        xyz="${a['mount_x']}  ${a['mount_y']} ${a['mount_z']}" rpy="0 0 ${a['mount_yaw']}"/>
+        xyz="${a['mount_x'] - pan_off * sin(a['left_yaw'])}  ${a['mount_y'] + pan_off * cos(a['left_yaw'])} ${a['mount_z']}"
+        rpy="0 0 ${a['left_yaw']}"/>
     <xacro:so101_arm prefix="right_arm" parent="base_link"
-        xyz="${a['mount_x']} ${-a['mount_y']} ${a['mount_z']}" rpy="0 0 ${a['mount_yaw']}"/>
+        xyz="${a['mount_x'] - pan_off * sin(a['right_yaw'])} ${-a['mount_y'] + pan_off * cos(a['right_yaw'])} ${a['mount_z']}"
+        rpy="0 0 ${a['right_yaw']}"/>
   </xacro:if>
   <xacro:if value="$(arg use_ros2_control)">
