Commit message: Measured heights: arm base 0.765, head junction 1.118, camera 1.183
Floor to the bottom of the arm base is 0.765 m (the arm base origin is its
bottom face). Floor to the top of the pan servo, where its axis meets the
printed part, is 1.118 m: in the upstream head meshes that junction is 0.073 m
above the pan joint origin, which puts the origin 0.325 m above the top base,
upstream has 0.323, so the neck is upstream's and needs no extension (a rod
is only added when the neck is more than 1 cm longer). The lens centre is
1.183 m, upstream's head puts it at 1.173, the camera mount z now follows the
measured value. The top base keeps its upstream position 0.045 m below the arm
surface.

Still the shared URDF's: the head shell is the depth-camera bar, the robot
has a plain USB camera, and the cart's position along the axle line.

File: src/xlerobot_description/urdf/head_pantilt.xacro (robot description, xacro)
@@ -14,9 +14,19 @@
   <xacro:macro name="xlerobot_head" params="dims parent">
     <xacro:property name="h" value="${dims['head']}"/>
-    <!-- top base sits 0.323 m below and 0.103 m ahead of the pan axis -->
+    <!-- The top base sits on the arm mounting surface, 0.045 m below it as in the
+         upstream URDF, and 0.103 m ahead of the pan axis. head: mount_z is the
+         measured height of the junction where the pan servo's axis meets the head's
+         printed part, that is 0.073 m above the pan joint origin in the upstream
+         head meshes, so the origin is at mount_z - 0.073. That gives 0.325 m above
+         the top base, upstream has 0.323. If the neck were longer than upstream's,
+         neck_ext is the difference and a plain rod fills it. -->
+    <xacro:property name="top_base_z" value="${dims['arms']['mount_z'] - 0.045}"/>
+    <xacro:property name="pan_z" value="${h['mount_z'] - 0.073}"/>
+    <xacro:property name="pan_dz" value="${pan_z - top_base_z}"/>
+    <xacro:property name="neck_ext" value="${pan_dz - 0.323}"/>
     <joint name="top_base_joint" type="fixed">
       <parent link="${parent}"/>
       <child link="top_base_link"/>
-      <origin xyz="${h['mount_x'] + 0.103} ${h['mount_y']} ${h['mount_z'] - 0.323}" rpy="0 0 0"/>
+      <origin xyz="${h['mount_x'] + 0.103} ${h['mount_y']} ${top_base_z}" rpy="0 0 0"/>
     </joint>
     <link name="top_base_link">
@@ -40,4 +50,11 @@
         <material name="xle_motor"/>
       </visual>
+      <xacro:if value="${neck_ext > 0.01}">
+        <visual>
+          <origin xyz="-0.103 0 ${0.323 + neck_ext / 2.0}" rpy="0 0 0"/>
+          <geometry><cylinder radius="0.03" length="${neck_ext}"/></geometry>
+          <material name="xle_motor"/>
+        </visual>
+      </xacro:if>
     </link>
     <link name="head_pan_link">
@@ -65,5 +82,5 @@
       <parent link="top_base_link"/>
       <child link="head_pan_link"/>
-      <origin xyz="-0.103 0 0.323" rpy="0 0 0"/>
+      <origin xyz="-0.103 0 ${pan_dz}" rpy="0 0 0"/>
       <axis xyz="0 0 1"/>
       <limit lower="${h['pan_limit_lower']}" upper="${h['pan_limit_upper']}" effort="2.0" velocity="3.0"/>
@@ -102,5 +119,6 @@
       <parent link="head_tilt_link"/>
       <child link="head_camera_mount"/>
-      <origin xyz="0.025 0 0.03" rpy="0 0 0"/>
+      <!-- z puts the lens centre at head: camera_z above the floor -->
+      <origin xyz="0.025 0 ${h['camera_z'] - pan_z - 0.09815}" rpy="0 0 0"/>
     </joint>
   </xacro:macro>

Commit message: Head camera shell of the plain USB camera instead of the depth camera bar

File: src/xlerobot_description/urdf/head_pantilt.xacro (robot description, xacro)
@@ -12,5 +12,5 @@
 -->
 <robot xmlns:xacro="http://www.ros.org/wiki/xacro">
-  <xacro:macro name="xlerobot_head" params="dims parent">
+  <xacro:macro name="xlerobot_head" params="dims parent sensor">
     <xacro:property name="h" value="${dims['head']}"/>
     <!-- The top base sits on the arm mounting surface, 0.045 m below it as in the
@@ -99,11 +99,15 @@
         <material name="xle_part"/>
       </visual>
-      <visual>
-        <origin xyz="0.16265 -0.006 -1.16815" rpy="0 0 0"/>
-        <geometry>
-          <mesh filename="package://xlerobot_description/meshes/upstream/tophead6.stl" scale="0.001 0.001 0.001"/>
-        </geometry>
-        <material name="xle_motor"/>
-      </visual>
+      <!-- tophead6 is the bar for the depth cameras, the plain USB camera has its own
+           shell, see sensors.xacro -->
+      <xacro:unless value="${sensor == 'usbcam'}">
+        <visual>
+          <origin xyz="0.16265 -0.006 -1.16815" rpy="0 0 0"/>
+          <geometry>
+            <mesh filename="package://xlerobot_description/meshes/upstream/tophead6.stl" scale="0.001 0.001 0.001"/>
+          </geometry>
+          <material name="xle_motor"/>
+        </visual>
+      </xacro:unless>
     </link>
     <joint name="head_tilt_joint" type="revolute">

File: src/xlerobot_description/urdf/sensors.xacro (robot description, xacro)
@@ -10,11 +10,15 @@
   <xacro:macro name="xlerobot_sensors" params="sensor dims">
     <!-- The head camera the robot has today: a plain USB webcam, the same model
-         as the wrist cameras (bringup cameras:=true, config/cameras.yaml). Body
-         size and pose on the head are approximate, not measured. -->
+         as the wrist cameras (bringup cameras:=true, config/cameras.yaml). The shell
+         is the printed one from the XLeRobot 3mf, placed with its lens hole centre on
+         head_camera_link, whose position is the measured lens centre. -->
     <xacro:if value="${sensor == 'usbcam'}">
       <link name="head_camera_link">
         <visual>
-          <geometry><box size="0.02 0.05 0.03"/></geometry>
-          <material name="xle_black"/>
+          <origin xyz="-0.0115 0 -0.0094" rpy="0 0 0"/>
+          <geometry>
+            <mesh filename="package://xlerobot_description/meshes/upstream/head_camera_shell.stl" scale="0.001 0.001 0.001"/>
+          </geometry>
+          <material name="xle_part"/>
         </visual>
         <inertial>

Commit message: Arm and head model zero and direction from the servo calibration
arms.joints and head.*_zero_step/_direction in robot_dimensions.yaml set the
driver's position_center_steps, and reverse the model's joint axis and mirror the
limits where the servo runs the other way. Calibration files of this robot as
examples.

File: src/xlerobot_description/urdf/head_pantilt.xacro (robot description, xacro)
@@ -83,6 +83,6 @@
       <child link="head_pan_link"/>
       <origin xyz="-0.103 0 ${pan_dz}" rpy="0 0 0"/>
-      <axis xyz="0 0 1"/>
-      <limit lower="${h['pan_limit_lower']}" upper="${h['pan_limit_upper']}" effort="2.0" velocity="3.0"/>
+      <axis xyz="0 0 ${-h['pan_direction']}"/>
+      <limit lower="${min(-h['pan_direction'] * h['pan_limit_lower'], -h['pan_direction'] * h['pan_limit_upper'])}" upper="${max(-h['pan_direction'] * h['pan_limit_lower'], -h['pan_direction'] * h['pan_limit_upper'])}" effort="2.0" velocity="3.0"/>
     </joint>
     <link name="head_tilt_link">
@@ -115,6 +115,6 @@
       <child link="head_tilt_link"/>
       <origin xyz="0.001 0.002 0.09815" rpy="0 0 3.1415927"/>
-      <axis xyz="0 1 0"/>
-      <limit lower="${h['tilt_limit_lower']}" upper="${h['tilt_limit_upper']}" effort="2.0" velocity="3.0"/>
+      <axis xyz="0 ${-h['tilt_direction']} 0"/>
+      <limit lower="${min(-h['tilt_direction'] * h['tilt_limit_lower'], -h['tilt_direction'] * h['tilt_limit_upper'])}" upper="${max(-h['tilt_direction'] * h['tilt_limit_lower'], -h['tilt_direction'] * h['tilt_limit_upper'])}" effort="2.0" velocity="3.0"/>
     </joint>
     <!-- sensor gets attached here, in sensors.xacro -->

File: src/xlerobot_description/urdf/so101_arm.xacro (robot description, xacro)
@@ -7,5 +7,7 @@
   stretched straight out to the side, and it folds by about +3 rad at the shoulder
   lift and elbow, which is how the real arms rest. Only the joint velocity limit
-  changed, the source has 0, 3 rad/s here so planners get a usable limit.
+  changed, the source has 0, 3 rad/s here so planners get a usable limit. Joint axes and
+  limits follow arms.joints in robot_dimensions.yaml: where the real servo goes the other
+  way from the source's angle the axis is reversed and the limits mirrored.
   Frame names follow the ros2_control joints and the sim, not upstream's
   (upstream calls the arm on the right side *_L). The wrist camera is upstream's
@@ -17,5 +19,26 @@
 -->
 <robot xmlns:xacro="http://www.ros.org/wiki/xacro">
-  <xacro:macro name="so101_arm" params="prefix parent xyz rpy wrist_camera:=true">
+  <xacro:macro name="so101_arm" params="prefix parent xyz rpy joints wrist_camera:=true">
+    <!-- joint direction, see arms.joints in robot_dimensions.yaml: m is -1 to reverse the
+         axis (and mirror the limits) where the servo step goes the same way as the joint
+         angle. Reversing axis and angle together is the same pose. -->
+    <xacro:property name="m_pan" value="${-joints['shoulder_pan']['direction']}"/>
+    <xacro:property name="lo_pan" value="${min(m_pan * joints['shoulder_pan']['lower'], m_pan * joints['shoulder_pan']['upper'])}"/>
+    <xacro:property name="hi_pan" value="${max(m_pan * joints['shoulder_pan']['lower'], m_pan * joints['shoulder_pan']['upper'])}"/>
+    <xacro:property name="m_lift" value="${-joints['shoulder_lift']['direction']}"/>
+    <xacro:property name="lo_lift" value="${min(m_lift * joints['shoulder_lift']['lower'], m_lift * joints['shoulder_lift']['upper'])}"/>
+    <xacro:property name="hi_lift" value="${max(m_lift * joints['shoulder_lift']['lower'], m_lift * joints['shoulder_lift']['upper'])}"/>
+    <xacro:property name="m_elbow" value="${-joints['elbow_flex']['direction']}"/>
+    <xacro:property name="lo_elbow" value="${min(m_elbow * joints['elbow_flex']['lower'], m_elbow * joints['elbow_flex']['upper'])}"/>
+    <xacro:property name="hi_elbow" value="${max(m_elbow * joints['elbow_flex']['lower'], m_elbow * joints['elbow_flex']['upper'])}"/>
+    <xacro:property name="m_wflex" value="${-joints['wrist_flex']['direction']}"/>
+    <xacro:property name="lo_wflex" value="${min(m_wflex * joints['wrist_flex']['lower'], m_wflex * joints['wrist_flex']['upper'])}"/>
+    <xacro:property name="hi_wflex" value="${max(m_wflex * joints['wrist_flex']['lower'], m_wflex * joints['wrist_flex']['upper'])}"/>
+    <xacro:property name="m_roll" value="${-joints['wrist_roll']['direction']}"/>
+    <xacro:property name="lo_roll" value="${min(m_roll * joints['wrist_roll']['lower'], m_roll * joints['wrist_roll']['upper'])}"/>
+    <xacro:property name="hi_roll" value="${max(m_roll * joints['wrist_roll']['lower'], m_roll * joints['wrist_roll']['upper'])}"/>
+    <xacro:property name="m_grip" value="${-joints['gripper']['direction']}"/>
+    <xacro:property name="lo_grip" value="${min(m_grip * joints['gripper']['lower'], m_grip * joints['gripper']['upper'])}"/>
+    <xacro:property name="hi_grip" value="${max(m_grip * joints['gripper']['lower'], m_grip * joints['gripper']['upper'])}"/>
     <joint name="${prefix}_mount_joint" type="fixed">
       <parent link="${parent}"/>
@@ -257,6 +280,6 @@
       <child link="${prefix}_shoulder_link"/>
       <origin xyz="0 -0.0452 0.0165" rpy="1.5708 0 0"/>
-      <axis xyz="0 -1 0"/>
-      <limit lower="-2.16" upper="2.16" effort="3.35" velocity="3.0"/>
+      <axis xyz="0 ${-1 * m_pan} 0"/>
+      <limit lower="${lo_pan}" upper="${hi_pan}" effort="3.35" velocity="3.0"/>
       <dynamics damping="0.6" friction="0.052"/>
     </joint>
@@ -265,6 +288,6 @@
       <child link="${prefix}_upper_arm_link"/>
       <origin xyz="0 0.1025 0.0306" rpy="1.5708 0 0"/>
-      <axis xyz="-1 0 0"/>
-      <limit lower="-0.22" upper="3.37" effort="3.35" velocity="3.0"/>
+      <axis xyz="${-1 * m_lift} 0 0"/>
+      <limit lower="${lo_lift}" upper="${hi_lift}" effort="3.35" velocity="3.0"/>
       <dynamics damping="0.6" friction="0.052"/>
     </joint>
@@ -273,6 +296,6 @@
       <child link="${prefix}_lower_arm_link"/>
       <origin xyz="0 0.11257 0.028" rpy="-1.5708 0 0"/>
-      <axis xyz="1 0 0"/>
-      <limit lower="-0.22" upper="3.14" effort="3.35" velocity="3.0"/>
+      <axis xyz="${m_elbow} 0 0"/>
+      <limit lower="${lo_elbow}" upper="${hi_elbow}" effort="3.35" velocity="3.0"/>
       <dynamics damping="0.6" friction="0.052"/>
     </joint>
@@ -281,6 +304,6 @@
       <child link="${prefix}_wrist_link"/>
       <origin xyz="0 0.0052 0.1349" rpy="-1.5708 0 0"/>
-      <axis xyz="1 0 0"/>
-      <limit lower="-1.6580628" upper="1.6580627" effort="3.35" velocity="3.0"/>
+      <axis xyz="${m_wflex} 0 0"/>
+      <limit lower="${lo_wflex}" upper="${hi_wflex}" effort="3.35" velocity="3.0"/>
       <dynamics damping="0.6" friction="0.052"/>
     </joint>
@@ -289,6 +312,6 @@
       <child link="${prefix}_gripper_link"/>
       <origin xyz="0 -0.0601 0" rpy="0 1.5707927 0"/>
-      <axis xyz="0 -1 0"/>
-      <limit lower="-2.7438473" upper="2.8412063" effort="3.35" velocity="3.0"/>
+      <axis xyz="0 ${-1 * m_roll} 0"/>
+      <limit lower="${lo_roll}" upper="${hi_roll}" effort="3.35" velocity="3.0"/>
       <dynamics damping="0.6" friction="0.052"/>
     </joint>
@@ -297,6 +320,6 @@
       <child link="${prefix}_moving_jaw_link"/>
       <origin xyz="-0.0202 -0.0244 0" rpy="3.1415854 -0.0000014 2.9531853"/>
-      <axis xyz="0 0 1"/>
-      <limit lower="-0.374533" upper="1.7453292" effort="10" velocity="3.0"/>
+      <axis xyz="0 0 ${m_grip}"/>
+      <limit lower="${lo_grip}" upper="${hi_grip}" effort="10" velocity="3.0"/>
       <dynamics damping="0.6" friction="0.052"/>
     </joint>

File: src/xlerobot_description/urdf/xlerobot.ros2_control.xacro (robot description, xacro)
@@ -29,8 +29,10 @@
   <!-- read_only: no command interface, so the driver disables torque on the joint and
        never writes to it, while its state is still read every cycle. -->
-  <xacro:macro name="sts_position_joint" params="name id lower upper read_only:=false">
+  <xacro:macro name="sts_position_joint" params="name id lower upper center:=4095 read_only:=false">
     <joint name="${name}">
       <param name="motor_id">${id}</param>
       <param name="operating_mode">0</param>
+      <!-- servo step that is 0 rad, the driver reports (center - step) -->
+      <param name="position_center_steps">${center}</param>
       <xacro:unless value="${read_only}">
         <command_interface name="position">
@@ -48,13 +50,21 @@
     </joint>
   </xacro:macro>
-  <!-- The six joints of one arm, IDs 1-6. Names and limits match so101_arm.xacro,
-       which has the limits of the arm in upstream's URDF. -->
-  <xacro:macro name="sts_arm_joints" params="prefix read_only">
-    <xacro:sts_position_joint name="${prefix}_shoulder_pan_joint"  id="1" lower="-2.16"      upper="2.16" read_only="${read_only}"/>
-    <xacro:sts_position_joint name="${prefix}_shoulder_lift_joint" id="2" lower="-0.22"      upper="3.37" read_only="${read_only}"/>
-    <xacro:sts_position_joint name="${prefix}_elbow_flex_joint"    id="3" lower="-0.22"      upper="3.14" read_only="${read_only}"/>
-    <xacro:sts_position_joint name="${prefix}_wrist_flex_joint"    id="4" lower="-1.6580628" upper="1.6580627" read_only="${read_only}"/>
-    <xacro:sts_position_joint name="${prefix}_wrist_roll_joint"    id="5" lower="-2.7438473" upper="2.8412063" read_only="${read_only}"/>
-    <xacro:sts_position_joint name="${prefix}_gripper_joint"       id="6" lower="-0.374533" upper="1.7453292" read_only="${read_only}"/>
+  <!-- One arm joint. The limits and the centre come from arms.joints in robot_dimensions.yaml
+       and match so101_arm.xacro: with direction +1 the model's joint is reversed against the
+       source URDF, so the limits are mirrored. -->
+  <xacro:macro name="sts_arm_joint" params="name id j read_only">
+    <xacro:property name="m" value="${-j['direction']}"/>
+    <xacro:sts_position_joint name="${name}" id="${id}"
+        lower="${min(m * j['lower'], m * j['upper'])}" upper="${max(m * j['lower'], m * j['upper'])}"
+        center="${j['zero_step']}" read_only="${read_only}"/>
+  </xacro:macro>
+  <!-- The six joints of one arm, IDs 1-6, names as in so101_arm.xacro. -->
+  <xacro:macro name="sts_arm_joints" params="prefix read_only joints">
+    <xacro:sts_arm_joint name="${prefix}_shoulder_pan_joint"  id="1" j="${joints['shoulder_pan']}"  read_only="${read_only}"/>
+    <xacro:sts_arm_joint name="${prefix}_shoulder_lift_joint" id="2" j="${joints['shoulder_lift']}" read_only="${read_only}"/>
+    <xacro:sts_arm_joint name="${prefix}_elbow_flex_joint"    id="3" j="${joints['elbow_flex']}"    read_only="${read_only}"/>
+    <xacro:sts_arm_joint name="${prefix}_wrist_flex_joint"    id="4" j="${joints['wrist_flex']}"    read_only="${read_only}"/>
+    <xacro:sts_arm_joint name="${prefix}_wrist_roll_joint"    id="5" j="${joints['wrist_roll']}"    read_only="${read_only}"/>
+    <xacro:sts_arm_joint name="${prefix}_gripper_joint"       id="6" j="${joints['gripper']}"       read_only="${read_only}"/>
   </xacro:macro>
   <xacro:macro name="xlerobot_ros2_control" params="bus1_port bus2_port use_mock_hardware with_arms torque_off with_head dims">
@@ -77,13 +87,17 @@
         </hardware>
         <xacro:if value="${with_arms}">
-          <xacro:sts_arm_joints prefix="left_arm" read_only="${torque_off}"/>
+          <xacro:sts_arm_joints prefix="left_arm" read_only="${torque_off}" joints="${dims['arms']['joints']}"/>
         </xacro:if>
         <xacro:if value="${with_head}">
+          <xacro:property name="pm" value="${-h['pan_direction']}"/>
+          <xacro:property name="tm" value="${-h['tilt_direction']}"/>
           <xacro:sts_position_joint name="head_pan_joint"  id="7"
-                                    lower="${h['pan_limit_lower']}"  upper="${h['pan_limit_upper']}"
-                                    read_only="${torque_off}"/>
+              lower="${min(pm * h['pan_limit_lower'], pm * h['pan_limit_upper'])}"
+              upper="${max(pm * h['pan_limit_lower'], pm * h['pan_limit_upper'])}"
+              center="${h['pan_zero_step']}" read_only="${torque_off}"/>
           <xacro:sts_position_joint name="head_tilt_joint" id="8"
-                                    lower="${h['tilt_limit_lower']}" upper="${h['tilt_limit_upper']}"
-                                    read_only="${torque_off}"/>
+              lower="${min(tm * h['tilt_limit_lower'], tm * h['tilt_limit_upper'])}"
+              upper="${max(tm * h['tilt_limit_lower'], tm * h['tilt_limit_upper'])}"
+              center="${h['tilt_zero_step']}" read_only="${torque_off}"/>
         </xacro:if>
       </ros2_control>
@@ -98,5 +112,5 @@
       </hardware>
       <xacro:if value="${with_arms}">
-        <xacro:sts_arm_joints prefix="right_arm" read_only="${torque_off}"/>
+        <xacro:sts_arm_joints prefix="right_arm" read_only="${torque_off}" joints="${dims['arms']['joints']}"/>
       </xacro:if>
       <!-- The RIGHT motor is mounted mirrored (confirmed on the real robot by

File: src/xlerobot_description/urdf/xlerobot.urdf.xacro (robot description, xacro)
@@ -60,8 +60,8 @@
     <xacro:property name="a" value="${dims['arms']}"/>
     <xacro:property name="pan_off" value="0.0452"/>
-    <xacro:so101_arm prefix="left_arm"  parent="body_link"
+    <xacro:so101_arm prefix="left_arm"  parent="body_link" joints="${a['joints']}"
         xyz="${a['mount_x'] - pan_off * sin(a['left_yaw'])} ${-a['mount_y'] + pan_off * cos(a['left_yaw'])} ${a['mount_z']}"
         rpy="0 0 ${a['left_yaw']}"/>
-    <xacro:so101_arm prefix="right_arm" parent="body_link"
+    <xacro:so101_arm prefix="right_arm" parent="body_link" joints="${a['joints']}"
         xyz="${a['mount_x'] - pan_off * sin(a['right_yaw'])}  ${a['mount_y'] + pan_off * cos(a['right_yaw'])} ${a['mount_z']}"
         rpy="0 0 ${a['right_yaw']}"/>
