Commit message: MoveIt 2 for the arms, arms in the Isaac twin
xlerobot_moveit_config: groups, named states, pick_ik position-only for the five joint arms,
controllers, generated self-collision matrix (tools/generate_moveit_collisions.py), launch file.
Collision geometry for the top base, head, camera and lidar. Rest and folded poses in
robot_dimensions.yaml. The Isaac scene builder takes its joints from the import URDF and starts
the arms in the rest pose. tools/moveit_smoke_test.py plans and executes on both arms.

File: src/xlerobot_description/urdf/head_pantilt.xacro (robot description, xacro)
@@ -43,4 +43,10 @@
         <material name="xle_part"/>
       </visual>
+      <collision>
+        <origin xyz="-0.44 -0.005 -0.6" rpy="0 0 0"/>
+        <geometry>
+          <mesh filename="package://xlerobot_description/meshes/upstream/topbase1.stl" scale="0.001 0.001 0.001"/>
+        </geometry>
+      </collision>
       <visual>
         <origin xyz="-0.298 0.006 -0.715" rpy="0 0 3.14"/>
@@ -50,4 +56,10 @@
         <material name="xle_motor"/>
       </visual>
+      <collision>
+        <origin xyz="-0.298 0.006 -0.715" rpy="0 0 3.14"/>
+        <geometry>
+          <mesh filename="package://xlerobot_description/meshes/upstream/topbase2.stl" scale="0.001 0.001 0.001"/>
+        </geometry>
+      </collision>
       <xacro:if value="${neck_ext > 0.01}">
         <visual>
@@ -56,4 +68,8 @@
           <material name="xle_motor"/>
         </visual>
+      <collision>
+          <origin xyz="-0.103 0 ${0.323 + neck_ext / 2.0}" rpy="0 0 0"/>
+          <geometry><cylinder radius="0.03" length="${neck_ext}"/></geometry>
+        </collision>
       </xacro:if>
     </link>
@@ -71,4 +87,10 @@
         <material name="xle_part"/>
       </visual>
+      <collision>
+        <origin xyz="-0.335 -0.005 -0.923" rpy="0 0 0"/>
+        <geometry>
+          <mesh filename="package://xlerobot_description/meshes/upstream/tophead1.stl" scale="0.001 0.001 0.001"/>
+        </geometry>
+      </collision>
       <visual>
         <origin xyz="1.17 -0.009 0.262" rpy="-3.141592 -1.57 -3.141592"/>
@@ -78,4 +100,10 @@
         <material name="xle_motor"/>
       </visual>
+      <collision>
+        <origin xyz="1.17 -0.009 0.262" rpy="-3.141592 -1.57 -3.141592"/>
+        <geometry>
+          <mesh filename="package://xlerobot_description/meshes/upstream/tophead4.stl" scale="0.001 0.001 0.001"/>
+        </geometry>
+      </collision>
     </link>
     <joint name="head_pan_joint" type="revolute">
@@ -99,4 +127,10 @@
         <material name="xle_part"/>
       </visual>
+      <collision>
+        <origin xyz="0.16265 -0.006 -1.16815" rpy="0 0 0"/>
+        <geometry>
+          <mesh filename="package://xlerobot_description/meshes/upstream/tophead5.stl" scale="0.001 0.001 0.001"/>
+        </geometry>
+      </collision>
       <!-- tophead6 is the bar for the depth cameras, the plain USB camera has its own
            shell, see sensors.xacro -->
@@ -109,4 +143,10 @@
           <material name="xle_motor"/>
         </visual>
+      <collision>
+          <origin xyz="0.16265 -0.006 -1.16815" rpy="0 0 0"/>
+          <geometry>
+            <mesh filename="package://xlerobot_description/meshes/upstream/tophead6.stl" scale="0.001 0.001 0.001"/>
+          </geometry>
+        </collision>
       </xacro:unless>
     </link>

File: src/xlerobot_description/urdf/lidar.xacro (robot description, xacro)
@@ -18,4 +18,10 @@
         <material name="xle_black"/>
       </visual>
+      <collision>
+        <!-- housing is 0.0349 m tall, its mounting surface is l['scan_below_mount'] above
+             the scan plane, that is at z = -scan_below_mount in this flipped frame -->
+        <origin xyz="0 0 ${-l['scan_below_mount'] + 0.0349 / 2}" rpy="0 0 0"/>
+        <geometry><cylinder radius="0.0193" length="0.0349"/></geometry>
+      </collision>
       <inertial>
         <mass value="0.047"/>

File: src/xlerobot_description/urdf/sensors.xacro (robot description, xacro)
@@ -22,4 +22,10 @@
           <material name="xle_part"/>
         </visual>
+      <collision>
+          <origin xyz="-0.0115 0 -0.0094" rpy="0 0 0"/>
+          <geometry>
+            <mesh filename="package://xlerobot_description/meshes/upstream/head_camera_shell.stl" scale="0.001 0.001 0.001"/>
+          </geometry>
+        </collision>
         <inertial>
           <mass value="0.03"/>
@@ -46,4 +52,7 @@
           <material name="xle_black"/>
         </visual>
+      <collision>
+          <geometry><box size="0.025 0.090 0.025"/></geometry>
+        </collision>
         <inertial>
           <mass value="0.072"/>
@@ -72,4 +81,7 @@
           <material name="xle_black"/>
         </visual>
+      <collision>
+          <geometry><box size="0.035 0.165 0.030"/></geometry>
+        </collision>
         <inertial>
           <mass value="0.12"/>
@@ -103,4 +115,7 @@
           <material name="xle_black"/>
         </visual>
+      <collision>
+          <geometry><cylinder radius="0.0516" length="0.0717"/></geometry>
+        </collision>
         <inertial>
           <mass value="0.83"/>

File: src/xlerobot_description/urdf/xlerobot.ros2_control_sim.xacro (robot description, xacro)
@@ -115,16 +115,16 @@
       <xacro:sim_position_joint name="head_tilt_joint"/>
       <xacro:if value="${with_arms}">
-        <xacro:sim_position_joint name="left_arm_shoulder_pan_joint"/>
-        <xacro:sim_position_joint name="left_arm_shoulder_lift_joint"/>
-        <xacro:sim_position_joint name="left_arm_elbow_flex_joint"/>
-        <xacro:sim_position_joint name="left_arm_wrist_flex_joint"/>
-        <xacro:sim_position_joint name="left_arm_wrist_roll_joint"/>
-        <xacro:sim_position_joint name="left_arm_gripper_joint"/>
-        <xacro:sim_position_joint name="right_arm_shoulder_pan_joint"/>
-        <xacro:sim_position_joint name="right_arm_shoulder_lift_joint"/>
-        <xacro:sim_position_joint name="right_arm_elbow_flex_joint"/>
-        <xacro:sim_position_joint name="right_arm_wrist_flex_joint"/>
-        <xacro:sim_position_joint name="right_arm_wrist_roll_joint"/>
-        <xacro:sim_position_joint name="right_arm_gripper_joint"/>
+        <xacro:sim_position_joint name="left_arm_shoulder_pan_joint" initial_position="${dims['arms']['rest_pose']['shoulder_pan']}"/>
+        <xacro:sim_position_joint name="left_arm_shoulder_lift_joint" initial_position="${dims['arms']['rest_pose']['shoulder_lift']}"/>
+        <xacro:sim_position_joint name="left_arm_elbow_flex_joint" initial_position="${dims['arms']['rest_pose']['elbow_flex']}"/>
+        <xacro:sim_position_joint name="left_arm_wrist_flex_joint" initial_position="${dims['arms']['rest_pose']['wrist_flex']}"/>
+        <xacro:sim_position_joint name="left_arm_wrist_roll_joint" initial_position="${dims['arms']['rest_pose']['wrist_roll']}"/>
+        <xacro:sim_position_joint name="left_arm_gripper_joint" initial_position="${dims['arms']['rest_pose']['gripper']}"/>
+        <xacro:sim_position_joint name="right_arm_shoulder_pan_joint" initial_position="${dims['arms']['rest_pose']['shoulder_pan']}"/>
+        <xacro:sim_position_joint name="right_arm_shoulder_lift_joint" initial_position="${dims['arms']['rest_pose']['shoulder_lift']}"/>
+        <xacro:sim_position_joint name="right_arm_elbow_flex_joint" initial_position="${dims['arms']['rest_pose']['elbow_flex']}"/>
+        <xacro:sim_position_joint name="right_arm_wrist_flex_joint" initial_position="${dims['arms']['rest_pose']['wrist_flex']}"/>
+        <xacro:sim_position_joint name="right_arm_wrist_roll_joint" initial_position="${dims['arms']['rest_pose']['wrist_roll']}"/>
+        <xacro:sim_position_joint name="right_arm_gripper_joint" initial_position="${dims['arms']['rest_pose']['gripper']}"/>
       </xacro:if>
     </ros2_control>

Commit message: Add head controller, fix MoveIt tracking on real hardware
- sts_hardware_interface proportional-speed unit mismatch fix (raw
  steps/s vs rad/s in std::min) uncovered CONTROL_FAILED on real
  hardware; this is the fallout in this repo: loosened smoke-test
  tolerance to account for the servos' known I=0 steady-state
  deadband, dropped now-unneeded per-joint trajectory/goal tolerances
  from controllers.yaml (JTC default -1 is fine).
- head_pan/head_tilt: real ros2_control controller, MoveIt group,
  URDF velocity limit was hardcoded to 3.0 instead of reading
  max_velocity from robot_dimensions.yaml, rate_limit added to match
  arms.
- RViz: pin Velocity/Acceleration_Scaling_Factor to 1.0 and a sane
  Interactive Marker Size, matching MoveIt's real defaults instead of
  the internal helper node's fallbacks.
- torque_off now defaults to false (bringup is commandable out of the
  box, matching the arms-bringup doc's actual guidance).

File: src/xlerobot_description/urdf/head_pantilt.xacro (robot description, xacro)
@@ -112,5 +112,5 @@
       <origin xyz="-0.103 0 ${pan_dz}" rpy="0 0 0"/>
       <axis xyz="0 0 ${-h['pan_direction']}"/>
-      <limit lower="${min(-h['pan_direction'] * h['pan_limit_lower'], -h['pan_direction'] * h['pan_limit_upper'])}" upper="${max(-h['pan_direction'] * h['pan_limit_lower'], -h['pan_direction'] * h['pan_limit_upper'])}" effort="2.0" velocity="3.0"/>
+      <limit lower="${min(-h['pan_direction'] * h['pan_limit_lower'], -h['pan_direction'] * h['pan_limit_upper'])}" upper="${max(-h['pan_direction'] * h['pan_limit_lower'], -h['pan_direction'] * h['pan_limit_upper'])}" effort="2.0" velocity="${h['max_velocity']}"/>
     </joint>
     <link name="head_tilt_link">
@@ -156,5 +156,5 @@
       <origin xyz="0.001 0.002 0.09815" rpy="0 0 3.1415927"/>
       <axis xyz="0 ${-h['tilt_direction']} 0"/>
-      <limit lower="${min(-h['tilt_direction'] * h['tilt_limit_lower'], -h['tilt_direction'] * h['tilt_limit_upper'])}" upper="${max(-h['tilt_direction'] * h['tilt_limit_lower'], -h['tilt_direction'] * h['tilt_limit_upper'])}" effort="2.0" velocity="3.0"/>
+      <limit lower="${min(-h['tilt_direction'] * h['tilt_limit_lower'], -h['tilt_direction'] * h['tilt_limit_upper'])}" upper="${max(-h['tilt_direction'] * h['tilt_limit_lower'], -h['tilt_direction'] * h['tilt_limit_upper'])}" effort="2.0" velocity="${h['max_velocity']}"/>
     </joint>
     <!-- sensor gets attached here, in sensors.xacro -->

File: src/xlerobot_description/urdf/xlerobot.ros2_control.xacro (robot description, xacro)
@@ -104,9 +104,9 @@
               lower="${min(pm * h['pan_limit_lower'], pm * h['pan_limit_upper'])}"
               upper="${max(pm * h['pan_limit_lower'], pm * h['pan_limit_upper'])}"
-              center="${h['pan_zero_step']}" read_only="${torque_off}"/>
+              center="${h['pan_zero_step']}" rate_limit="${1.25 * h['max_velocity']}" read_only="${torque_off}"/>
           <xacro:sts_position_joint name="head_tilt_joint" id="8"
               lower="${min(tm * h['tilt_limit_lower'], tm * h['tilt_limit_upper'])}"
               upper="${max(tm * h['tilt_limit_lower'], tm * h['tilt_limit_upper'])}"
-              center="${h['tilt_zero_step']}" read_only="${torque_off}"/>
+              center="${h['tilt_zero_step']}" rate_limit="${1.25 * h['max_velocity']}" read_only="${torque_off}"/>
         </xacro:if>
       </ros2_control>

Commit message: Fix head_tilt_joint's axis sign - model pitched the wrong way vs reality
head_camera_optical_frame's computed orientation pitched UP for a negative
head_tilt_joint value, when the real hardware physically tilts DOWN for
the same value (confirmed on hardware: tilt=-0.385 rad visibly points the
camera at the desk, not the ceiling). Root cause: head_tilt_joint's
origin applies a 180 degree yaw flip (rpy="0 0 pi", inherited from
head_pan_link being turned around per this file's own top comment) before
the joint's own axis rotation is applied. That origin flip inverts the
effective sign of a same-axis rotation relative to the parent frame, and
the existing axis="0 ${-h['tilt_direction']} 0"} compensation didn't
account for it - a double negative that canceled out the intended fix,
so the already-correct tilt_direction=-1 value was applied with the wrong
overall sign for the final camera pitch specifically.

Does not touch tilt_limit_lower/upper, the servo-step zero_step/direction
hardware calibration, or any saved joint-radian values - this only
changes which spatial direction the model draws for a given joint value,
not what values the real hardware reports or accepts.

Verified on real hardware: regenerated the URDF with the fix, restarted
robot_state_publisher standalone (no hardware/torque impact) at the same
physical tilt=-0.385 rad position, confirmed head_camera_optical_frame's
forward axis Z-component flipped from +0.376 (model said "pointing up")
to -0.376 (now correctly "pointing down", matching physical reality).

This was caught because Rerun's 3D view visibly showed the head camera
frustum pointing up while it was physically pointing down at a desk -
Rerun was rendering the TF correctly, the TF itself was wrong.

Claude-Session: https://claude.ai/code/session_019BnndKspkjHQhoYCb9Cr5q

File: src/xlerobot_description/urdf/head_pantilt.xacro (robot description, xacro)
@@ -155,5 +155,5 @@
       <child link="head_tilt_link"/>
       <origin xyz="0.001 0.002 0.09815" rpy="0 0 3.1415927"/>
-      <axis xyz="0 ${-h['tilt_direction']} 0"/>
+      <axis xyz="0 ${h['tilt_direction']} 0"/>
       <limit lower="${min(-h['tilt_direction'] * h['tilt_limit_lower'], -h['tilt_direction'] * h['tilt_limit_upper'])}" upper="${max(-h['tilt_direction'] * h['tilt_limit_lower'], -h['tilt_direction'] * h['tilt_limit_upper'])}" effort="2.0" velocity="${h['max_velocity']}"/>
     </joint>
