Commit message: Make the Orbbec Gemini 2 the default head camera
Physically replaced the head usbcam with the Gemini 2 (3D-printed holder cut
flat, camera screwed to it). sensor:=gemini is now the default end to end:
xlerobot.urdf.xacro, threaded through bringup.launch.py, and cameras.launch.py
brings up orbbec_camera's gemini2.launch.py for "head" instead of usb_cam,
remapping color/image_raw and color/camera_info so existing flat-topic
consumers (MCP server, rerun_bridge) keep working, with depth/ir/point
cloud/IMU newly available at their native topic names.

Live-tested and fixed two real bugs along the way:
- camera_name:="cameras/head" can't double as a ROS2 node name (can't contain
  "/") - restructured to a stacked PushRosNamespace instead.
- the driver's extrinsic TF tree root is "<camera_name>_link", not a fixed
  "camera_link" as first assumed from a standalone test that left camera_name
  at its own default - and it's only published with
  enable_publish_extrinsic:=true, which the vendor launch file defaults to
  false. sensors.xacro and cameras.yaml's frame_id now match the real
  "head_link"/"head_color_optical_frame" names. Confirmed base_link ->
  head_color_optical_frame resolves end to end, color/depth streaming at
  ~22/~26Hz, and the MCP server's capture_image returns the right frame_id.

Also corrects ADR-0003/ARCHITECTURE.md's prior misidentification of the
camera as the original Gemini - it's a Gemini 2, confirmed via the device's
own firmware response through the vendor driver.

Claude-Session: https://claude.ai/code/session_019BnndKspkjHQhoYCb9Cr5q

File: src/xlerobot_description/urdf/sensors.xacro (robot description, xacro)
@@ -74,6 +74,27 @@
     </xacro:if>
     <xacro:if value="${sensor == 'gemini'}">
-      <!-- same mount point, different body size, see ADR-0003 for whether this
-           camera works on Jazzy at all -->
+      <!-- Orbbec Gemini 2 (confirmed via its own firmware + the vendor driver's device
+           table, 2026-10-05 - project docs previously misidentified this as the original
+           Gemini, see ADR-0003). Box size is a first-cut placeholder, not yet measured
+           against the real unit - refine once it's mounted and visible.
+           Unlike usbcam/realsense above, this link is NOT the camera's optical frame -
+           it's named head_camera_link (project convention for "sits on head_camera_mount")
+           but then connects, with identity rotation, to a second link named exactly
+           "head_link": the orbbec_camera driver (gemini2.launch.py) publishes its own
+           calibrated extrinsic TF tree rooted at "<camera_name>_link", not a fixed
+           "camera_link" as first assumed - confirmed live only after passing
+           camera_name:="head" (cameras.launch.py's actual invocation, needed for topic
+           naming), which renames every frame in the tree with that prefix: head_link ->
+           head_depth_frame -> head_{color,ir}_frame -> head_{color,ir}_optical_frame,
+           plus head_{accel,gyro}_frame/_optical_frame. An earlier standalone test left
+           camera_name at its own default ("camera"), which happened to render as
+           "camera_link" and looked like a hardcoded constant - it wasn't. So this URDF
+           only needs to place head_link at the right physical pose - the driver handles
+           every per-stream optical frame itself, unlike usbcam/realsense which need the
+           REP-103 remap done by hand below.
+           Identity rotation here is the first-cut assumption matching the camera's
+           physical mount (3D-printed holder cut down flat, camera sits horizontal,
+           forward axis assumed aligned with head_camera_mount's own forward axis) -
+           tune this rpy by hand once the real pointing direction is visible. -->
       <link name="head_camera_link">
         <visual>
@@ -94,9 +115,9 @@
         <origin xyz="0 0 0" rpy="0 0 0"/>
       </joint>
-      <link name="head_camera_optical_frame"/>
-      <joint name="head_camera_optical_joint" type="fixed">
+      <link name="head_link"/>
+      <joint name="head_link_joint" type="fixed">
         <parent link="head_camera_link"/>
-        <child  link="head_camera_optical_frame"/>
-        <origin xyz="0 0 0" rpy="${-pi/2} 0 ${-pi/2}"/>
+        <child  link="head_link"/>
+        <origin xyz="0 0 0" rpy="0 0 0"/>
       </joint>
     </xacro:if>

File: src/xlerobot_description/urdf/xlerobot.urdf.xacro (robot description, xacro)
@@ -21,7 +21,8 @@
   <xacro:arg name="bus1_port"         default="/dev/xle-bus1"/>
   <xacro:arg name="bus2_port"         default="/dev/xle-bus2"/>
-  <!-- none | usbcam | vlp16 | gemini | realsense, see ADR-0003. usbcam is the head
-       camera the robot has today. -->
-  <xacro:arg name="sensor"            default="usbcam"/>
+  <!-- none | usbcam | vlp16 | gemini | realsense, see ADR-0003. gemini (Orbbec Gemini 2)
+       is the head camera the robot has today - it physically replaced the usbcam
+       2026-10-05. -->
+  <xacro:arg name="sensor"            default="gemini"/>
   <!-- none | ld19, the 2D lidar under the second basket -->
   <xacro:arg name="lidar"             default="ld19"/>

Commit message: Pitch the Gemini mount 9.2 deg nose up
The camera's own IMU read 9.2 deg higher than the joints predicted at head tilt
0 and at -0.59 rad, and a flat ChArUco board on a desk agreed to about 1.5 deg.
With the correction the board normal is vertical to 0.1 deg in the base frame
and the board sits 8 mm from the measured desk height.

File: src/xlerobot_description/urdf/sensors.xacro (robot description, xacro)
@@ -93,8 +93,8 @@
            every per-stream optical frame itself, unlike usbcam/realsense which need the
            REP-103 remap done by hand below.
-           Identity rotation here is the first-cut assumption matching the camera's
-           physical mount (3D-printed holder cut down flat, camera sits horizontal,
-           forward axis assumed aligned with head_camera_mount's own forward axis) -
-           tune this rpy by hand once the real pointing direction is visible. -->
+           Pitch is -0.1606 rad (9.2 deg nose up), from the camera's own IMU: with the head
+           tilt at 0 and at -0.59 rad it read 9.2 deg higher than the joints predicted both
+           times, and a flat ChArUco board agrees to about 1.5 deg. Roll (about 1 deg) and
+           yaw are left at 0. -->
       <link name="head_camera_link">
         <visual>
@@ -113,5 +113,5 @@
         <parent link="head_camera_mount"/>
         <child  link="head_camera_link"/>
-        <origin xyz="0 0 0" rpy="0 0 0"/>
+        <origin xyz="0 0 0" rpy="0 -0.1606 0"/>
       </joint>
       <link name="head_link"/>
